Commit message: Fixed
1. math needs to be wrapped in a single ${} see ${ 1 + 2 * radius + x}
2.  cos(radius) makes no sense, it isnt defined. Should be theta
3. were some extra parans in there

File: urdf/test.urdf.xacro (robot description, xacro)
@@ -54,5 +54,5 @@
         <parent link="base_link"/>
         <child link="right_roller_${prefix}"/>
-        <origin xyz="$(cos(radius))*$(roller_radius) $(roller_side_length) $(cos(radius))*$(roller_radius*)" rpy="0 theta 0"/>
+        <origin xyz="${cos(theta)*roller_radius} ${roller_side_length} ${cos(theta)*roller_radius}" rpy="0 theta 0"/>
     </joint>
 </xacro:macro>

Commit message: quick fix

File: urdf/test.urdf.xacro (robot description, xacro)
@@ -54,8 +54,10 @@
         <parent link="base_link"/>
         <child link="right_roller_${prefix}"/>
-        <origin xyz="${cos(theta)*roller_radius} ${roller_side_length} ${cos(theta)*roller_radius}" rpy="0 theta 0"/>
+        <origin xyz="${cos(theta)*roller_radius} ${roller_side_length} ${cos(theta)*roller_radius}" rpy="0 ${theta} 0"/>
     </joint>
 </xacro:macro>
 <xacro:right_roller prefix="one" theta="0"/>
+<xacro:right_roller prefix="two" theta="${pi / 4}"/>
+<xacro:right_roller prefix="three" theta="${3*pi / 4}"/>
 <!--
 -->

Commit message: no

File: urdf/test.urdf.xacro (robot description, xacro)
@@ -13,4 +13,12 @@
   <color rgba="1 1 1 1"/>
 </material>
+<xacro:macro name="default_inertial" params="mass">
+	<inertial>
+     		<mass value="${mass}" />
+	        <inertia ixx="1.0" ixy="0.0" ixz="0.0"
+            		           iyy="1.0" iyz="0.0"
+                                         izz="1.0" />
+	</inertial>
+</xacro:macro>
 <link name="base_link">
     <visual>
@@ -27,4 +35,5 @@
         <origin xyz="${xyz}" rpy="${rpy}"/>
     </collision>
+    <xacro:default_inertial mass="1"/>
 </link>
 <!--offset from the center of the wheel for the rollers-->
@@ -50,4 +59,5 @@
             <origin xyz="0 0 0" rpy="0 0 0"/>
         </collision>
+        <xacro:default_inertial mass="1"/>
     </link>
     <joint name="joint_to_right_roller_${prefix}" type="fixed">

Commit message: :zap: IT WORKS!!

File: urdf/test.urdf.xacro (robot description, xacro)
@@ -40,5 +40,5 @@
 <xacro:property name="roller_side_length" value=".0055"/>
 <!--radius where the rollers are placed-->
-<xacro:property name="roller_radius" value=".01"/>
+<xacro:property name="roller_radius" value=".049"/>
 <!--This is for all of the right rollers. I made a way to send theta to
 calculate the x, y, z, and pitch based off of parameters listed directly
@@ -61,14 +61,23 @@
         <xacro:default_inertial mass="1"/>
     </link>
-    <joint name="joint_to_right_roller_${prefix}" type="fixed">
+    <joint name="joint_to_right_roller_${prefix}" type="continuous">
         <parent link="base_link"/>
         <child link="right_roller_${prefix}"/>
-        <origin xyz="${cos(theta)*roller_radius} ${roller_side_length} ${cos(theta)*roller_radius}" rpy="0 ${theta} 0"/>
+        <!--<origin xyz="0 0 0" rpy="0 0 0"/>-->
+        <origin xyz="${sin(theta)*roller_radius} 0 ${cos(theta)*roller_radius}" rpy="0 ${theta + pi/2} 0"/><!---->
     </joint>
 </xacro:macro>
-<xacro:right_roller prefix="one" theta="0"/>
-<xacro:right_roller prefix="two" theta="${pi / 4}"/>
-<xacro:right_roller prefix="three" theta="${3*pi / 4}"/>
-<!--
+<xacro:right_roller prefix="one" theta="${pi * ( 1/6)}"/>
+<xacro:right_roller prefix="two" theta="${pi * ( 2/6)}"/>
+<xacro:right_roller prefix="thr" theta="${pi * ( 3/6)}"/>
+<xacro:right_roller prefix="for" theta="${pi * ( 4/6)}"/>
+<xacro:right_roller prefix="fve" theta="${pi * ( 5/6)}"/>
+<xacro:right_roller prefix="six" theta="${pi * ( 6/6)}"/>
+<xacro:right_roller prefix="svn" theta="${pi * ( 7/6)}"/>
+<xacro:right_roller prefix="ate" theta="${pi * ( 8/6)}"/>
+<xacro:right_roller prefix="nne" theta="${pi * ( 9/6)}"/>
+<xacro:right_roller prefix="ten" theta="${pi * (10/6)}"/>
+<xacro:right_roller prefix="lvn" theta="${pi * (11/6)}"/>
+<xacro:right_roller prefix="wlv" theta="${pi * (12/6)}"/>
 -->
 </robot>

Commit message: :white_check_mark: omni wheel done (joint is still weird)

File: urdf/test.urdf.xacro (robot description, xacro)
@@ -44,6 +44,6 @@
 calculate the x, y, z, and pitch based off of parameters listed directly
 above-->
-<xacro:macro name="right_roller" params="prefix theta">
-    <link name="right_roller_${prefix}">
+<xacro:macro name="roller" params="prefix theta side">
+    <link name="roller_${prefix}">
         <visual>
             <geometry>
@@ -63,21 +63,33 @@
     <joint name="joint_to_right_roller_${prefix}" type="continuous">
         <parent link="base_link"/>
-        <child link="right_roller_${prefix}"/>
-        <!--<origin xyz="0 0 0" rpy="0 0 0"/>-->
-        <origin xyz="${sin(theta)*roller_radius} 0 ${cos(theta)*roller_radius}" rpy="0 ${theta + pi/2} 0"/><!---->
+        <child link="roller_${prefix}"/>
+        <!--<limit lower="$(-2000 * pi)" upper="$(2000 * pi)" effort="0" velocity="1"/>-->
+        <!--this math may not be correct-->
+        <origin xyz="${sin(theta)*roller_radius} ${roller_side_length*side} ${cos(theta)*roller_radius}" rpy="0 ${theta + pi/2} 0"/><!---->
     </joint>
 </xacro:macro>
-<xacro:right_roller prefix="one" theta="${pi * ( 1/6)}"/>
-<xacro:right_roller prefix="two" theta="${pi * ( 2/6)}"/>
-<xacro:right_roller prefix="thr" theta="${pi * ( 3/6)}"/>
-<xacro:right_roller prefix="for" theta="${pi * ( 4/6)}"/>
-<xacro:right_roller prefix="fve" theta="${pi * ( 5/6)}"/>
-<xacro:right_roller prefix="six" theta="${pi * ( 6/6)}"/>
-<xacro:right_roller prefix="svn" theta="${pi * ( 7/6)}"/>
-<xacro:right_roller prefix="ate" theta="${pi * ( 8/6)}"/>
-<xacro:right_roller prefix="nne" theta="${pi * ( 9/6)}"/>
-<xacro:right_roller prefix="ten" theta="${pi * (10/6)}"/>
-<xacro:right_roller prefix="lvn" theta="${pi * (11/6)}"/>
-<xacro:right_roller prefix="wlv" theta="${pi * (12/6)}"/>
--->
+<xacro:roller prefix="right_one" theta="${pi * ( 1/6)}" side="1"/>
+<xacro:roller prefix="right_two" theta="${pi * ( 2/6)}" side="1"/>
+<xacro:roller prefix="right_thr" theta="${pi * ( 3/6)}" side="1"/>
+<xacro:roller prefix="right_for" theta="${pi * ( 4/6)}" side="1"/>
+<xacro:roller prefix="right_fve" theta="${pi * ( 5/6)}" side="1"/>
+<xacro:roller prefix="right_six" theta="${pi * ( 6/6)}" side="1"/>
+<xacro:roller prefix="right_svn" theta="${pi * ( 7/6)}" side="1"/>
+<xacro:roller prefix="right_ate" theta="${pi * ( 8/6)}" side="1"/>
+<xacro:roller prefix="right_nne" theta="${pi * ( 9/6)}" side="1"/>
+<xacro:roller prefix="right_ten" theta="${pi * (10/6)}" side="1"/>
+<xacro:roller prefix="right_lvn" theta="${pi * (11/6)}" side="1"/>
+<xacro:roller prefix="right_wlv" theta="${pi * (12/6)}" side="1"/>
+<xacro:roller prefix="left_one" theta="${pi * ( 1/6) + ( pi / 12 )}" side="-1"/>
+<xacro:roller prefix="left_two" theta="${pi * ( 2/6) + ( pi / 12 )}" side="-1"/>
+<xacro:roller prefix="left_thr" theta="${pi * ( 3/6) + ( pi / 12 )}" side="-1"/>
+<xacro:roller prefix="left_for" theta="${pi * ( 4/6) + ( pi / 12 )}" side="-1"/>
+<xacro:roller prefix="left_fve" theta="${pi * ( 5/6) + ( pi / 12 )}" side="-1"/>
+<xacro:roller prefix="left_six" theta="${pi * ( 6/6) + ( pi / 12 )}" side="-1"/>
+<xacro:roller prefix="left_svn" theta="${pi * ( 7/6) + ( pi / 12 )}" side="-1"/>
+<xacro:roller prefix="left_ate" theta="${pi * ( 8/6) + ( pi / 12 )}" side="-1"/>
+<xacro:roller prefix="left_nne" theta="${pi * ( 9/6) + ( pi / 12 )}" side="-1"/>
+<xacro:roller prefix="left_ten" theta="${pi * (10/6) + ( pi / 12 )}" side="-1"/>
+<xacro:roller prefix="left_lvn" theta="${pi * (11/6) + ( pi / 12 )}" side="-1"/>
+<xacro:roller prefix="left_wlv" theta="${pi * (12/6) + ( pi / 12 )}" side="-1"/>
 </robot>

Commit message: rollers make sense now

File: urdf/test.urdf.xacro (robot description, xacro)
@@ -50,5 +50,5 @@
               <cylinder radius="${roller_diameter}" length="${roller_width}"/>
             </geometry>
-            <origin xyz="0 0 0" rpy="0 0 0"/>
+            <origin xyz="0 0 0" rpy="0 ${pi/2} 0"/>
             <material name="white"/>
         </visual>
@@ -57,5 +57,5 @@
               <cylinder radius="${roller_diameter}" length="${roller_width}"/>
             </geometry>
-            <origin xyz="0 0 0" rpy="0 0 0"/>
+            <origin xyz="0 0 0" rpy="0 ${pi/2} 0"/>
         </collision>
         <xacro:default_inertial mass="1"/>
@@ -66,5 +66,5 @@
         <!--<limit lower="$(-2000 * pi)" upper="$(2000 * pi)" effort="0" velocity="1"/>-->
         <!--this math may not be correct-->
-        <origin xyz="${sin(theta)*roller_radius} ${roller_side_length*side} ${cos(theta)*roller_radius}" rpy="0 ${theta + pi/2} 0"/><!---->
+        <origin xyz="${sin(theta)*roller_radius} ${roller_side_length*side} ${cos(theta)*roller_radius}" rpy="0 ${theta} 0"/><!---->
     </joint>
 </xacro:macro>

Commit message: no

File: urdf/test.urdf.xacro (robot description, xacro)
@@ -50,5 +50,6 @@
               <cylinder radius="${roller_diameter}" length="${roller_width}"/>
             </geometry>
-            <origin xyz="0 0 0" rpy="0 0 0"/>
+            <!--this math may not be correct-->
+            <origin xyz="0 0 0" rpy="0 ${theta + pi/2} 0"/><!---->
             <material name="white"/>
         </visual>
@@ -57,5 +58,6 @@
               <cylinder radius="${roller_diameter}" length="${roller_width}"/>
             </geometry>
-            <origin xyz="0 0 0" rpy="0 0 0"/>
+            <!--this math may not be correct-->
+            <origin xyz="0 0 0" rpy="0 ${theta + pi/2} 0"/><!---->
         </collision>
         <xacro:default_inertial mass="1"/>
@@ -64,7 +66,8 @@
         <parent link="base_link"/>
         <child link="roller_${prefix}"/>
-        <!--<limit lower="$(-2000 * pi)" upper="$(2000 * pi)" effort="0" velocity="1"/>-->
-        <!--this math may not be correct-->
-        <origin xyz="${sin(theta)*roller_radius} ${roller_side_length*side} ${cos(theta)*roller_radius}" rpy="0 ${theta + pi/2} 0"/><!---->
+<!--        <origin xyz="${sin(theta)*roller_radius} ${roller_side_length*side} ${cos(theta)*roller_radius}" rpy="0 0 0">
+-->        <axis xyz="0 1 0" rpy="0  0" />
+        <limit effort="100" velocity="100"/>
+        <joint_properties damping="0.0" friction="0.0"/>
     </joint>
 </xacro:macro>

Commit message: :ambulance: omni wheel fix

File: urdf/test.urdf.xacro (robot description, xacro)
@@ -4,5 +4,7 @@
 <xacro:property name="wheel_width" value="0.025" />
 <xacro:property name="xyz" value="0 0 0"/>
-<xacro:property name="rpy" value="1.5708 0 0"/>
+<xacro:property name="rpy" value="0 0 0"/>
+<xacro:property name="roller_xyz" value="0 .008 -.0465"/>
+<xacro:property name="roller_rpy" value="0 ${-pi/12} 0"/>
 <xacro:property name="roller_diameter" value="0.0055" />
 <xacro:property name="roller_width" value="0.015" />
@@ -24,5 +26,5 @@
     <visual>
         <geometry>
-            <cylinder radius="${wheel_radius}" length="${wheel_width}"/>
+            <mesh filename="package://gazebosim/gazeboSimulation/models/VexRobot/OmniWheelNoRollers.stl"/>
         </geometry>
         <origin xyz="${xyz}" rpy="${rpy}"/>
@@ -31,5 +33,5 @@
     <collision>
         <geometry>
-            <cylinder radius="${wheel_radius}" length="${wheel_width}"/>
+            <mesh filename="package://gazebosim/gazeboSimulation/models/VexRobot/OmniWheelNoRollers.stl"/>
         </geometry>
         <origin xyz="${xyz}" rpy="${rpy}"/>
@@ -40,5 +42,5 @@
 <xacro:property name="roller_side_length" value=".0055"/>
 <!--radius where the rollers are placed-->
-<xacro:property name="roller_radius" value=".049"/>
+<xacro:property name="roller_radius" value=".0465"/>
 <!--This is for all of the right rollers. I made a way to send theta to
 calculate the x, y, z, and pitch based off of parameters listed directly
@@ -48,14 +50,14 @@
         <visual>
             <geometry>
-              <cylinder radius="${roller_diameter}" length="${roller_width}"/>
+                <mesh filename="package://gazebosim/gazeboSimulation/models/VexRobot/Roller.stl"/>
             </geometry>
-            <origin xyz="0 0 0" rpy="0 ${pi/2} 0"/>
+            <origin xyz="${roller_xyz}" rpy="${roller_rpy}"/>
             <material name="white"/>
         </visual>
         <collision>
             <geometry>
-              <cylinder radius="${roller_diameter}" length="${roller_width}"/>
+                <mesh filename="package://gazebosim/gazeboSimulation/models/VexRobot/Roller.stl"/>
             </geometry>
-            <origin xyz="0 0 0" rpy="0 ${pi/2} 0"/>
+            <origin xyz="${roller_xyz}" rpy="${roller_rpy}"/>
         </collision>
         <xacro:default_inertial mass="1"/>
@@ -64,5 +66,4 @@
         <parent link="base_link"/>
         <child link="roller_${prefix}"/>
-        <!--<limit lower="$(-2000 * pi)" upper="$(2000 * pi)" effort="0" velocity="1"/>-->
         <!--this math may not be correct-->
         <origin xyz="${sin(theta)*roller_radius} ${roller_side_length*side} ${cos(theta)*roller_radius}" rpy="0 ${theta} 0"/><!---->
@@ -93,3 +94,5 @@
 <xacro:roller prefix="left_lvn" theta="${pi * (11/6) + ( pi / 12 )}" side="-1"/>
 <xacro:roller prefix="left_wlv" theta="${pi * (12/6) + ( pi / 12 )}" side="-1"/>
+<!--
+-->
 </robot>

Commit message: :dizzy: umm. last couple bugs

File: urdf/test.urdf.xacro (robot description, xacro)
@@ -5,10 +5,22 @@
 <xacro:property name="xyz" value="0 0 0"/>
 <xacro:property name="rpy" value="0 0 0"/>
+<xacro:property name="wheel_xyz" value="0 0 0"/>
+<xacro:property name="wheel_rpy" value="0 0 0"/>
 <xacro:property name="roller_xyz" value="0 .008 -.0465"/>
 <xacro:property name="roller_rpy" value="0 ${-pi/12} 0"/>
 <xacro:property name="roller_diameter" value="0.0055" />
 <xacro:property name="roller_width" value="0.015" />
+<!--offset from the center of the wheel for the rollers-->
+<xacro:property name="roller_side_length" value=".0055"/>
+<!--radius where the rollers are placed-->
+<xacro:property name="roller_radius" value=".0465"/>
 <material name="blue">
-  <color rgba="0 0 0.8 1"/>
+  <color rgba="0 0 .8 1"/>
+</material>
+<material name="grey">
+  <color rgba=".18 .19 .19 1"/>
+</material>
+<material name="silver">
+  <color rgba=".5176 .5294 .5373 1"/>
 </material>
 <material name="white">
@@ -26,26 +38,19 @@
     <visual>
         <geometry>
-            <mesh filename="package://gazebosim/gazeboSimulation/models/VexRobot/OmniWheelNoRollers.stl"/>
+            <box size=".3048 .3048 .0254"/>
         </geometry>
-        <origin xyz="${xyz}" rpy="${rpy}"/>
-        <material name="blue"/>
+        <origin xyz="0 0 0" rpy="0 0 0"/>
+        <material name="silver"/>
     </visual>
     <collision>
         <geometry>
-            <mesh filename="package://gazebosim/gazeboSimulation/models/VexRobot/OmniWheelNoRollers.stl"/>
+            <mesh filename="package://gazebosim/gazeboSimulation/models/VexRobot/chassis.dae"/>
         </geometry>
-        <origin xyz="${xyz}" rpy="${rpy}"/>
+        <origin xyz="0 0 0" rpy="0 0 0"/>
     </collision>
     <xacro:default_inertial mass="1"/>
 </link>
-<!--offset from the center of the wheel for the rollers-->
-<xacro:property name="roller_side_length" value=".0055"/>
-<!--radius where the rollers are placed-->
-<xacro:property name="roller_radius" value=".0465"/>
-<!--This is for all of the right rollers. I made a way to send theta to
-calculate the x, y, z, and pitch based off of parameters listed directly
-above-->
-<xacro:macro name="roller" params="prefix theta side">
-    <link name="roller_${prefix}">
+<xacro:macro name="roller" params="prefix suffix theta side changeInX changeInY">
+    <link name="${prefix}_roller_${suffix}">
         <visual>
             <geometry>
@@ -63,35 +68,61 @@
         <xacro:default_inertial mass="1"/>
     </link>
-    <joint name="joint_to_right_roller_${prefix}" type="continuous">
+    <joint name="joint_to_${prefix}_roller_${suffix}" type="continuous">
         <parent link="base_link"/>
-        <child link="roller_${prefix}"/>
-        <!--this math may not be correct-->
-        <origin xyz="${sin(theta)*roller_radius} ${roller_side_length*side} ${cos(theta)*roller_radius}" rpy="0 ${theta} 0"/><!---->
+        <child link="${prefix}_roller_${suffix}"/>
+        <origin xyz="${sin(theta)*roller_radius-changeInY} ${roller_side_length*side+changeInX} ${cos(theta)*roller_radius}" rpy="0 ${theta} 0"/>
     </joint>
 </xacro:macro>
-<xacro:roller prefix="right_one" theta="${pi * ( 1/6)}" side="1"/>
-<xacro:roller prefix="right_two" theta="${pi * ( 2/6)}" side="1"/>
-<xacro:roller prefix="right_thr" theta="${pi * ( 3/6)}" side="1"/>
-<xacro:roller prefix="right_for" theta="${pi * ( 4/6)}" side="1"/>
-<xacro:roller prefix="right_fve" theta="${pi * ( 5/6)}" side="1"/>
-<xacro:roller prefix="right_six" theta="${pi * ( 6/6)}" side="1"/>
-<xacro:roller prefix="right_svn" theta="${pi * ( 7/6)}" side="1"/>
-<xacro:roller prefix="right_ate" theta="${pi * ( 8/6)}" side="1"/>
-<xacro:roller prefix="right_nne" theta="${pi * ( 9/6)}" side="1"/>
-<xacro:roller prefix="right_ten" theta="${pi * (10/6)}" side="1"/>
-<xacro:roller prefix="right_lvn" theta="${pi * (11/6)}" side="1"/>
-<xacro:roller prefix="right_wlv" theta="${pi * (12/6)}" side="1"/>
-<xacro:roller prefix="left_one" theta="${pi * ( 1/6) + ( pi / 12 )}" side="-1"/>
-<xacro:roller prefix="left_two" theta="${pi * ( 2/6) + ( pi / 12 )}" side="-1"/>
-<xacro:roller prefix="left_thr" theta="${pi * ( 3/6) + ( pi / 12 )}" side="-1"/>
-<xacro:roller prefix="left_for" theta="${pi * ( 4/6) + ( pi / 12 )}" side="-1"/>
-<xacro:roller prefix="left_fve" theta="${pi * ( 5/6) + ( pi / 12 )}" side="-1"/>
-<xacro:roller prefix="left_six" theta="${pi * ( 6/6) + ( pi / 12 )}" side="-1"/>
-<xacro:roller prefix="left_svn" theta="${pi * ( 7/6) + ( pi / 12 )}" side="-1"/>
-<xacro:roller prefix="left_ate" theta="${pi * ( 8/6) + ( pi / 12 )}" side="-1"/>
-<xacro:roller prefix="left_nne" theta="${pi * ( 9/6) + ( pi / 12 )}" side="-1"/>
-<xacro:roller prefix="left_ten" theta="${pi * (10/6) + ( pi / 12 )}" side="-1"/>
-<xacro:roller prefix="left_lvn" theta="${pi * (11/6) + ( pi / 12 )}" side="-1"/>
-<xacro:roller prefix="left_wlv" theta="${pi * (12/6) + ( pi / 12 )}" side="-1"/>
+<xacro:macro name="wheel" params="prefix changeInX changeInY">
+    <link name="wheel_${prefix}">
+        <visual>
+            <geometry>
+                <mesh filename="package://gazebosim/gazeboSimulation/models/VexRobot/OmniWheelNoRollers.stl"/>
+            </geometry>
+            <origin xyz="0 0 0" rpy="0 0 0"/>
+            <material name="blue"/>
+        </visual>
+        <collision>
+            <geometry>
+                <mesh filename="package://gazebosim/gazeboSimulation/models/VexRobot/OmniWheelNoRollers.stl"/>
+            </geometry>
+            <origin xyz="0 0 0" rpy="0 0 0"/>
+        </collision>
+        <xacro:default_inertial mass="1"/>
+    </link>
+    <joint name="joint_to_wheel_${prefix}" type="continuous">
+        <parent link="base_link"/>
+        <child link="wheel_${prefix}"/>
+        <origin xyz="${-changeInY} ${changeInX} 0" rpy="0 0 0"/>
+    </joint>
+    <xacro:roller prefix="${prefix}" suffix="right_one" theta="${pi * ( 1/6)}" side="1" changeInX="${changeInX}" changeInY="${changeInY}"/>
+    <xacro:roller prefix="${prefix}" suffix="right_two" theta="${pi * ( 2/6)}" side="1" changeInX="${changeInX}" changeInY="${changeInY}"/>
+    <xacro:roller prefix="${prefix}" suffix="right_thr" theta="${pi * ( 3/6)}" side="1" changeInX="${changeInX}" changeInY="${changeInY}"/>
+    <xacro:roller prefix="${prefix}" suffix="right_for" theta="${pi * ( 4/6)}" side="1" changeInX="${changeInX}" changeInY="${changeInY}"/>
+    <xacro:roller prefix="${prefix}" suffix="right_fve" theta="${pi * ( 5/6)}" side="1" changeInX="${changeInX}" changeInY="${changeInY}"/>
+    <xacro:roller prefix="${prefix}" suffix="right_six" theta="${pi * ( 6/6)}" side="1" changeInX="${changeInX}" changeInY="${changeInY}"/>
+    <xacro:roller prefix="${prefix}" suffix="right_svn" theta="${pi * ( 7/6)}" side="1" changeInX="${changeInX}" changeInY="${changeInY}"/>
+    <xacro:roller prefix="${prefix}" suffix="right_ate" theta="${pi * ( 8/6)}" side="1" changeInX="${changeInX}" changeInY="${changeInY}"/>
+    <xacro:roller prefix="${prefix}" suffix="right_nne" theta="${pi * ( 9/6)}" side="1" changeInX="${changeInX}" changeInY="${changeInY}"/>
+    <xacro:roller prefix="${prefix}" suffix="right_ten" theta="${pi * (10/6)}" side="1" changeInX="${changeInX}" changeInY="${changeInY}"/>
+    <xacro:roller prefix="${prefix}" suffix="right_lvn" theta="${pi * (11/6)}" side="1" changeInX="${changeInX}" changeInY="${changeInY}"/>
+    <xacro:roller prefix="${prefix}" suffix="right_wlv" theta="${pi * (12/6)}" side="1" changeInX="${changeInX}" changeInY="${changeInY}"/>
+    <xacro:roller prefix="${prefix}" suffix="left_one" theta="${pi * ( 1/6) + ( pi / 12 )}" side="-1" changeInX="${changeInX}" changeInY="${changeInY}"/>
+    <xacro:roller prefix="${prefix}" suffix="left_two" theta="${pi * ( 2/6) + ( pi / 12 )}" side="-1" changeInX="${changeInX}" changeInY="${changeInY}"/>
+    <xacro:roller prefix="${prefix}" suffix="left_thr" theta="${pi * ( 3/6) + ( pi / 12 )}" side="-1" changeInX="${changeInX}" changeInY="${changeInY}"/>
+    <xacro:roller prefix="${prefix}" suffix="left_for" theta="${pi * ( 4/6) + ( pi / 12 )}" side="-1" changeInX="${changeInX}" changeInY="${changeInY}"/>
+    <xacro:roller prefix="${prefix}" suffix="left_fve" theta="${pi * ( 5/6) + ( pi / 12 )}" side="-1" changeInX="${changeInX}" changeInY="${changeInY}"/>
+    <xacro:roller prefix="${prefix}" suffix="left_six" theta="${pi * ( 6/6) + ( pi / 12 )}" side="-1" changeInX="${changeInX}" changeInY="${changeInY}"/>
+    <xacro:roller prefix="${prefix}" suffix="left_svn" theta="${pi * ( 7/6) + ( pi / 12 )}" side="-1" changeInX="${changeInX}" changeInY="${changeInY}"/>
+    <xacro:roller prefix="${prefix}" suffix="left_ate" theta="${pi * ( 8/6) + ( pi / 12 )}" side="-1" changeInX="${changeInX}" changeInY="${changeInY}"/>
+    <xacro:roller prefix="${prefix}" suffix="left_nne" theta="${pi * ( 9/6) + ( pi / 12 )}" side="-1" changeInX="${changeInX}" changeInY="${changeInY}"/>
+    <xacro:roller prefix="${prefix}" suffix="left_ten" theta="${pi * (10/6) + ( pi / 12 )}" side="-1" changeInX="${changeInX}" changeInY="${changeInY}"/>
+    <xacro:roller prefix="${prefix}" suffix="left_lvn" theta="${pi * (11/6) + ( pi / 12 )}" side="-1" changeInX="${changeInX}" changeInY="${changeInY}"/>
+    <xacro:roller prefix="${prefix}" suffix="left_wlv" theta="${pi * (12/6) + ( pi / 12 )}" side="-1" changeInX="${changeInX}" changeInY="${changeInY}"/>
+</xacro:macro>
+<xacro:wheel prefix="front_right" changeInX=" .17145" changeInY=" .10145"/>
+<xacro:wheel prefix="front_left " changeInX="-.17145" changeInY=" .10145"/>
+<xacro:wheel prefix="back_right " changeInX=" .17145" changeInY="-.10145"/>
+<xacro:wheel prefix="back_left  " changeInX="-.17145" changeInY="-.10145"/>
 <!--
 -->
