Commit message: :bug: fixed roller joint

File: urdf/test.urdf.xacro (robot description, xacro)
@@ -51,5 +51,5 @@
     <xacro:default_inertial mass="1"/>
 </link>
-<xacro:macro name="roller" params="prefix suffix theta side changeInX changeInY">
+<xacro:macro name="roller" params="prefix suffix theta side">
     <link name="${prefix}_roller_${suffix}">
         <visual>
@@ -69,7 +69,7 @@
     </link>
     <joint name="joint_to_${prefix}_roller_${suffix}" type="continuous">
-        <parent link="base_link"/>
+        <parent link="wheel_${prefix}"/>
         <child link="${prefix}_roller_${suffix}"/>
-        <origin xyz="${sin(theta)*roller_radius-changeInY} ${roller_side_length*side+changeInX} ${cos(theta)*roller_radius}" rpy="0 ${theta} 0"/>
+        <origin xyz="${sin(theta)*roller_radius} ${roller_side_length*side} ${cos(theta)*roller_radius}" rpy="0 ${theta} 0"/>
     </joint>
 </xacro:macro>
@@ -94,30 +94,30 @@
         <parent link="base_link"/>
         <child link="wheel_${prefix}"/>
-        <origin xyz="${-changeInY} ${changeInX} 0" rpy="0 0 0"/>
+        <origin xyz="${-changeInY} ${changeInX} 0" rpy="0 ${pi/2} 0"/>
     </joint>
-    <xacro:roller prefix="${prefix}" suffix="right_one" theta="${pi * ( 1/6)}" side="1" changeInX="${changeInX}" changeInY="${changeInY}"/>
-    <xacro:roller prefix="${prefix}" suffix="right_two" theta="${pi * ( 2/6)}" side="1" changeInX="${changeInX}" changeInY="${changeInY}"/>
-    <xacro:roller prefix="${prefix}" suffix="right_thr" theta="${pi * ( 3/6)}" side="1" changeInX="${changeInX}" changeInY="${changeInY}"/>
-    <xacro:roller prefix="${prefix}" suffix="right_for" theta="${pi * ( 4/6)}" side="1" changeInX="${changeInX}" changeInY="${changeInY}"/>
-    <xacro:roller prefix="${prefix}" suffix="right_fve" theta="${pi * ( 5/6)}" side="1" changeInX="${changeInX}" changeInY="${changeInY}"/>
-    <xacro:roller prefix="${prefix}" suffix="right_six" theta="${pi * ( 6/6)}" side="1" changeInX="${changeInX}" changeInY="${changeInY}"/>
-    <xacro:roller prefix="${prefix}" suffix="right_svn" theta="${pi * ( 7/6)}" side="1" changeInX="${changeInX}" changeInY="${changeInY}"/>
-    <xacro:roller prefix="${prefix}" suffix="right_ate" theta="${pi * ( 8/6)}" side="1" changeInX="${changeInX}" changeInY="${changeInY}"/>
-    <xacro:roller prefix="${prefix}" suffix="right_nne" theta="${pi * ( 9/6)}" side="1" changeInX="${changeInX}" changeInY="${changeInY}"/>
-    <xacro:roller prefix="${prefix}" suffix="right_ten" theta="${pi * (10/6)}" side="1" changeInX="${changeInX}" changeInY="${changeInY}"/>
-    <xacro:roller prefix="${prefix}" suffix="right_lvn" theta="${pi * (11/6)}" side="1" changeInX="${changeInX}" changeInY="${changeInY}"/>
-    <xacro:roller prefix="${prefix}" suffix="right_wlv" theta="${pi * (12/6)}" side="1" changeInX="${changeInX}" changeInY="${changeInY}"/>
-    <xacro:roller prefix="${prefix}" suffix="left_one" theta="${pi * ( 1/6) + ( pi / 12 )}" side="-1" changeInX="${changeInX}" changeInY="${changeInY}"/>
-    <xacro:roller prefix="${prefix}" suffix="left_two" theta="${pi * ( 2/6) + ( pi / 12 )}" side="-1" changeInX="${changeInX}" changeInY="${changeInY}"/>
-    <xacro:roller prefix="${prefix}" suffix="left_thr" theta="${pi * ( 3/6) + ( pi / 12 )}" side="-1" changeInX="${changeInX}" changeInY="${changeInY}"/>
-    <xacro:roller prefix="${prefix}" suffix="left_for" theta="${pi * ( 4/6) + ( pi / 12 )}" side="-1" changeInX="${changeInX}" changeInY="${changeInY}"/>
-    <xacro:roller prefix="${prefix}" suffix="left_fve" theta="${pi * ( 5/6) + ( pi / 12 )}" side="-1" changeInX="${changeInX}" changeInY="${changeInY}"/>
-    <xacro:roller prefix="${prefix}" suffix="left_six" theta="${pi * ( 6/6) + ( pi / 12 )}" side="-1" changeInX="${changeInX}" changeInY="${changeInY}"/>
-    <xacro:roller prefix="${prefix}" suffix="left_svn" theta="${pi * ( 7/6) + ( pi / 12 )}" side="-1" changeInX="${changeInX}" changeInY="${changeInY}"/>
-    <xacro:roller prefix="${prefix}" suffix="left_ate" theta="${pi * ( 8/6) + ( pi / 12 )}" side="-1" changeInX="${changeInX}" changeInY="${changeInY}"/>
-    <xacro:roller prefix="${prefix}" suffix="left_nne" theta="${pi * ( 9/6) + ( pi / 12 )}" side="-1" changeInX="${changeInX}" changeInY="${changeInY}"/>
-    <xacro:roller prefix="${prefix}" suffix="left_ten" theta="${pi * (10/6) + ( pi / 12 )}" side="-1" changeInX="${changeInX}" changeInY="${changeInY}"/>
-    <xacro:roller prefix="${prefix}" suffix="left_lvn" theta="${pi * (11/6) + ( pi / 12 )}" side="-1" changeInX="${changeInX}" changeInY="${changeInY}"/>
-    <xacro:roller prefix="${prefix}" suffix="left_wlv" theta="${pi * (12/6) + ( pi / 12 )}" side="-1" changeInX="${changeInX}" changeInY="${changeInY}"/>
+    <xacro:roller prefix="${prefix}" suffix="right_one" theta="${pi * ( 1/6)}" side="1"/>
+    <xacro:roller prefix="${prefix}" suffix="right_two" theta="${pi * ( 2/6)}" side="1"/>
+    <xacro:roller prefix="${prefix}" suffix="right_thr" theta="${pi * ( 3/6)}" side="1"/>
+    <xacro:roller prefix="${prefix}" suffix="right_for" theta="${pi * ( 4/6)}" side="1"/>
+    <xacro:roller prefix="${prefix}" suffix="right_fve" theta="${pi * ( 5/6)}" side="1"/>
+    <xacro:roller prefix="${prefix}" suffix="right_six" theta="${pi * ( 6/6)}" side="1"/>
+    <xacro:roller prefix="${prefix}" suffix="right_svn" theta="${pi * ( 7/6)}" side="1"/>
+    <xacro:roller prefix="${prefix}" suffix="right_ate" theta="${pi * ( 8/6)}" side="1"/>
+    <xacro:roller prefix="${prefix}" suffix="right_nne" theta="${pi * ( 9/6)}" side="1"/>
+    <xacro:roller prefix="${prefix}" suffix="right_ten" theta="${pi * (10/6)}" side="1"/>
+    <xacro:roller prefix="${prefix}" suffix="right_lvn" theta="${pi * (11/6)}" side="1"/>
+    <xacro:roller prefix="${prefix}" suffix="right_wlv" theta="${pi * (12/6)}" side="1"/>
+    <xacro:roller prefix="${prefix}" suffix="left_one" theta="${pi * ( 1/6) + ( pi / 12 )}" side="-1"/>
+    <xacro:roller prefix="${prefix}" suffix="left_two" theta="${pi * ( 2/6) + ( pi / 12 )}" side="-1"/>
+    <xacro:roller prefix="${prefix}" suffix="left_thr" theta="${pi * ( 3/6) + ( pi / 12 )}" side="-1"/>
+    <xacro:roller prefix="${prefix}" suffix="left_for" theta="${pi * ( 4/6) + ( pi / 12 )}" side="-1"/>
+    <xacro:roller prefix="${prefix}" suffix="left_fve" theta="${pi * ( 5/6) + ( pi / 12 )}" side="-1"/>
+    <xacro:roller prefix="${prefix}" suffix="left_six" theta="${pi * ( 6/6) + ( pi / 12 )}" side="-1"/>
+    <xacro:roller prefix="${prefix}" suffix="left_svn" theta="${pi * ( 7/6) + ( pi / 12 )}" side="-1"/>
+    <xacro:roller prefix="${prefix}" suffix="left_ate" theta="${pi * ( 8/6) + ( pi / 12 )}" side="-1"/>
+    <xacro:roller prefix="${prefix}" suffix="left_nne" theta="${pi * ( 9/6) + ( pi / 12 )}" side="-1"/>
+    <xacro:roller prefix="${prefix}" suffix="left_ten" theta="${pi * (10/6) + ( pi / 12 )}" side="-1"/>
+    <xacro:roller prefix="${prefix}" suffix="left_lvn" theta="${pi * (11/6) + ( pi / 12 )}" side="-1"/>
+    <xacro:roller prefix="${prefix}" suffix="left_wlv" theta="${pi * (12/6) + ( pi / 12 )}" side="-1"/>
 </xacro:macro>
 <xacro:wheel prefix="front_right" changeInX=" .17145" changeInY=" .10145"/>

Commit message: fix wheel rotation axis

File: urdf/test.urdf.xacro (robot description, xacro)
@@ -80,5 +80,5 @@
                 <mesh filename="package://gazebosim/gazeboSimulation/models/VexRobot/OmniWheelNoRollers.stl"/>
             </geometry>
-            <origin xyz="0 0 0" rpy="0 0 0"/>
+            <origin xyz="0 0 0" rpy="0 0 ${pi/2}"/>
             <material name="blue"/>
         </visual>
@@ -87,5 +87,5 @@
                 <mesh filename="package://gazebosim/gazeboSimulation/models/VexRobot/OmniWheelNoRollers.stl"/>
             </geometry>
-            <origin xyz="0 0 0" rpy="0 0 0"/>
+            <origin xyz="0 0 0" rpy="0 0 ${pi/2}"/>
         </collision>
         <xacro:default_inertial mass="1"/>
@@ -94,5 +94,5 @@
         <parent link="base_link"/>
         <child link="wheel_${prefix}"/>
-        <origin xyz="${-changeInY} ${changeInX} 0" rpy="0 ${pi/2} 0"/>
+        <origin xyz="${-changeInY} ${changeInX} 0" rpy="0 0 ${-pi/2}"/>
     </joint>
     <xacro:roller prefix="${prefix}" suffix="right_one" theta="${pi * ( 1/6)}" side="1"/>

Commit message: 95% fix rollers issue

File: urdf/test.urdf.xacro (robot description, xacro)
@@ -71,5 +71,5 @@
         <parent link="wheel_${prefix}"/>
         <child link="${prefix}_roller_${suffix}"/>
-        <origin xyz="${sin(theta)*roller_radius} ${roller_side_length*side} ${cos(theta)*roller_radius}" rpy="0 ${theta} 0"/>
+        <origin xyz="${roller_side_length*side} ${sin(theta)*roller_radius} ${cos(theta)*roller_radius}" rpy="${pi/2} ${theta} ${pi/2}"/>
     </joint>
 </xacro:macro>

Commit message: :sparkles: added transmission for wheels

File: urdf/test.urdf.xacro (robot description, xacro)
@@ -96,4 +96,14 @@
         <origin xyz="${-changeInY} ${changeInX} 0" rpy="0 0 ${-pi/2}"/>
     </joint>
+    <transmission name="transmission_to_wheel_${prefix}">
+      <type>transmission_interface/SimpleTransmission</type>
+      <joint name="joint_to_wheel_${prefix}">
+            <hardwareInterface>EffortJointInterface</hardwareInterface>
+      </joint>
+      <actuator name="motor_wheel_${prefix}">
+            <hardwareInterface>EffortJointInterface</hardwareInterface>
+            <mechanicalReduction>1</mechanicalReduction>
+      </actuator>
+    </transmission>
     <xacro:roller prefix="${prefix}" suffix="right_one" theta="${pi * ( 1/6)}" side="-1"/>
     <xacro:roller prefix="${prefix}" suffix="right_two" theta="${pi * ( 2/6)}" side="-1"/>
@@ -125,5 +135,8 @@
 <xacro:wheel prefix="back_right " changeInX=" .17145" changeInY="-.10145"/>
 <xacro:wheel prefix="back_left  " changeInX="-.17145" changeInY="-.10145"/>
-<!--
--->
+<gazebo>
+  <plugin name="gazebo_ros_control" filename="libgazebo_ros_control.so">
+    <robotNamespace>/</robotNamespace>
+  </plugin>
+</gazebo>
 </robot>
