Commit message: Completely remove dependency on deprecated repo

File: urdf/robot.urdf.xacro (robot description, xacro)
@@ -1,142 +1,172 @@
 <?xml version="1.0"?>
-<robot name="macroed" xmlns:xacro="http://ros.org/wiki/xacro">
-<xacro:property name="wheel_radius" value="0.04" />
-<xacro:property name="wheel_width" value="0.025" />
-<xacro:property name="xyz" value="0 0 0"/>
-<xacro:property name="rpy" value="0 0 0"/>
-<xacro:property name="wheel_xyz" value="0 0 0"/>
-<xacro:property name="wheel_rpy" value="0 0 0"/>
-<xacro:property name="roller_xyz" value="0 .008 -.0465"/>
-<xacro:property name="roller_rpy" value="0 ${-pi/12} 0"/>
-<xacro:property name="roller_diameter" value="0.0055" />
-<xacro:property name="roller_width" value="0.015" />
-<!--offset from the center of the wheel for the rollers-->
-<xacro:property name="roller_side_length" value=".0055"/>
-<!--radius where the rollers are placed-->
-<xacro:property name="roller_radius" value=".0465"/>
-<material name="blue">
-  <color rgba="0 0 .8 1"/>
-</material>
-<material name="grey">
-  <color rgba=".18 .19 .19 1"/>
-</material>
-<material name="silver">
-  <color rgba=".5176 .5294 .5373 1"/>
-</material>
-<material name="white">
-  <color rgba="1 1 1 1"/>
-</material>
-<xacro:macro name="default_inertial" params="mass">
-	<inertial>
-     		<mass value="${mass}" />
-	        <inertia ixx="1.0" ixy="0.0" ixz="0.0"
-            		           iyy="1.0" iyz="0.0"
-                                         izz="1.0" />
-	</inertial>
-</xacro:macro>
-<link name="base_link">
+<robot name="roscontrol" xmlns:xacro="http://ros.org/wiki/xacro">
+  <xacro:property name="width" value="0.1" />
+  <xacro:property name="leglen" value="0.05" />
+  <xacro:property name="bodylen" value="0.05" />
+  <xacro:property name="baselen" value="0.4" />
+  <xacro:property name="wheeldiam" value="0.082" />
+  <xacro:property name="pi" value="3.1415" />
+  <xacro:property name="wheel_radius" value="0.04" />
+  <xacro:property name="wheel_width" value="0.025" />
+  <xacro:property name="xyz" value="0 0 0"/>
+  <xacro:property name="rpy" value="0 0 0"/>
+  <xacro:property name="wheel_xyz" value="0 0 0"/>
+  <xacro:property name="wheel_rpy" value="0 0 0"/>
+  <xacro:property name="roller_xyz" value="0 .008 -.0465"/>
+  <xacro:property name="roller_rpy" value="0 ${-pi/12} 0"/>
+  <xacro:property name="roller_diameter" value="0.0055" />
+  <xacro:property name="roller_width" value="0.015" />
+  <xacro:property name="roller_side_length" value="0.0088"/>
+  <xacro:property name="roller_radius" value=".0475"/>
+  <material name="blue">
+    <color rgba="0 0 0.8 1"/>
+  </material>
+  <material name="black">
+    <color rgba="0 0 0 1"/>
+  </material>
+  <material name="white">
+    <color rgba="1 1 1 1"/>
+  </material>
+  <xacro:macro name="default_inertial" params="mass">
+    <inertial>
+      <mass value="${mass}" />
+      <inertia ixx="1.0" ixy="0.0" ixz="0.0" iyy="1.0" iyz="0.0" izz="1.0" />
+    </inertial>
+  </xacro:macro>
+  <link name="base_link">
     <visual>
-        <geometry>
-            <box size=".3048 .3048 .0254"/>
-        </geometry>
-        <origin xyz="0 0 0" rpy="0 0 0"/>
-        <material name="silver"/>
+      <geometry>
+        <cylinder radius="${width}" length="${bodylen}"/>
+      </geometry>
+      <material name="blue"/>
     </visual>
     <collision>
+      <geometry>
+        <cylinder radius="${width}" length="${bodylen}"/>
+      </geometry>
+    </collision>
+    <xacro:default_inertial mass="10"/>
+  </link>
+  <xacro:macro name="roller" params="prefix suffix theta side">
+    <link name="${prefix}_${suffix}_roller">
+      <visual>
+        <origin xyz="0 0 0" rpy="0 ${pi/2} 0" />
         <geometry>
-            <mesh filename="package://gazebosim/gazeboSimulation/models/VexRobot/chassis.dae"/>
+          <cylinder radius="${roller_diameter}" length="${roller_width}"/>
         </geometry>
-        <origin xyz="0 0 0" rpy="0 0 0"/>
-    </collision>
-    <xacro:default_inertial mass="1"/>
-</link>
-<xacro:macro name="roller" params="prefix suffix theta side">
-    <link name="${prefix}_roller_${suffix}">
-        <visual>
-            <geometry>
-                <mesh filename="package://gazebosim/gazeboSimulation/models/VexRobot/Roller.stl"/>
-            </geometry>
-            <origin xyz="${roller_xyz}" rpy="${roller_rpy}"/>
-            <material name="white"/>
-        </visual>
-        <collision>
-            <geometry>
-                <mesh filename="package://gazebosim/gazeboSimulation/models/VexRobot/Roller.stl"/>
-            </geometry>
-            <origin xyz="${roller_xyz}" rpy="${roller_rpy}"/>
-        </collision>
-        <xacro:default_inertial mass="1"/>
+        <material name="black"/>
+      </visual>
+      <collision>
+        <origin xyz="0 0 0" rpy="0 ${pi/2} 0" />
+        <geometry>
+          <cylinder radius="${roller_diameter}" length="${roller_width}"/>
+        </geometry>
+      </collision>
+      <xacro:default_inertial mass="1"/>
     </link>
-    <joint name="joint_to_${prefix}_roller_${suffix}" type="continuous">
-        <parent link="wheel_${prefix}"/>
-        <child link="${prefix}_roller_${suffix}"/>
-        <origin xyz="${roller_side_length*side} ${sin(theta)*roller_radius} ${cos(theta)*roller_radius}" rpy="${pi/2} ${theta} ${pi/2}"/>
+    <joint name="${prefix}_${suffix}_roller_joint" type="continuous">
+      <axis xyz="0 1 0" rpy="0 0 0" />
+      <parent link="${prefix}_wheel"/>
+      <child link="${prefix}_${suffix}_roller"/>
+      <origin xyz="${sin(theta)*roller_radius} ${roller_side_length*side} ${cos(theta)*roller_radius}" rpy="0 ${theta} 0"/>
     </joint>
-</xacro:macro>
-<xacro:macro name="wheel" params="prefix changeInX changeInY">
-    <link name="wheel_${prefix}">
-        <visual>
-            <geometry>
-                <mesh filename="package://gazebosim/gazeboSimulation/models/VexRobot/OmniWheelNoRollers.stl"/>
-            </geometry>
-            <origin xyz="0 0 0" rpy="0 0 ${pi/2}"/>
-            <material name="blue"/>
-        </visual>
-        <collision>
-            <geometry>
-                <mesh filename="package://gazebosim/gazeboSimulation/models/VexRobot/OmniWheelNoRollers.stl"/>
-            </geometry>
-            <origin xyz="0 0 0" rpy="0 0 ${pi/2}"/>
-        </collision>
-        <xacro:default_inertial mass="1"/>
+    <!-- This block provides the simulator (Gazebo) with information on a few additional
+    physical properties. See http://gazebosim.org/tutorials/?tut=ros_urdf for more-->
+    <gazebo reference="${prefix}_${suffix}_roller">
+      <mu1 value="200.0"/>
+      <mu2 value="100.0"/>
+      <kp value="10000000.0" />
+      <kd value="1.0" />
+      <material>Gazebo/Grey</material>
+    </gazebo>
+    <!-- This block connects the wheel joint to an actuator (motor), which informs both
+    simulation and visualization of the robot -->
+    <transmission name="${prefix}_${suffix}_roller_trans">
+      <type>transmission_interface/SimpleTransmission</type>
+      <actuator name="${prefix}_${suffix}_roller_motor">
+        <mechanicalReduction>1</mechanicalReduction>
+      </actuator>
+      <joint name="${prefix}_${suffix}_roller_joint">
+        <hardwareInterface>VelocityJointInterface</hardwareInterface>
+      </joint>
+    </transmission>
+  </xacro:macro>
+  <xacro:macro name="wheel" params="prefix suffix reflect reflectX">
+    <link name="${prefix}_${suffix}_wheel">
+      <visual>
+        <origin xyz="0 0 0" rpy="${pi/2} 0 0" />
+        <geometry>
+          <cylinder radius="${wheeldiam/2}" length="${wheel_width}"/>
+        </geometry>
+        <material name="black"/>
+      </visual>
+      <collision>
+        <origin xyz="0 0 0" rpy="${pi/2} 0 0" />
+        <geometry>
+          <cylinder radius="${wheeldiam/2}" length="${wheel_width}"/>
+        </geometry>
+      </collision>
+      <xacro:default_inertial mass="1"/>
     </link>
-    <joint name="joint_to_wheel_${prefix}" type="continuous">
-        <parent link="base_link"/>
-        <child link="wheel_${prefix}"/>
-        <origin xyz="${-changeInY} ${changeInX} 0" rpy="0 0 ${-pi/2}"/>
+    <joint name="${prefix}_${suffix}_wheel_joint" type="continuous">
+      <axis xyz="0 1 0" rpy="0 0 0" />
+      <parent link="base_link"/>
+      <child link="${prefix}_${suffix}_wheel"/>
+      <origin xyz="${baselen*reflect/3} ${.1*reflectX} -.05" rpy="0 0 0"/>
     </joint>
-    <transmission name="transmission_to_wheel_${prefix}">
+    <!-- This block provides the simulator (Gazebo) with information on a few additional
+    physical properties. See http://gazebosim.org/tutorials/?tut=ros_urdf for more-->
+    <gazebo reference="${prefix}_${suffix}_wheel">
+      <mu1 value="200.0"/>
+      <mu2 value="100.0"/>
+      <kp value="10000000.0" />
+      <kd value="1.0" />
+      <material>Gazebo/Grey</material>
+    </gazebo>
+    <!-- This block connects the wheel joint to an actuator (motor), which informs both
+    simulation and visualization of the robot -->
+    <transmission name="${prefix}_${suffix}_wheel_trans">
       <type>transmission_interface/SimpleTransmission</type>
-      <joint name="joint_to_wheel_${prefix}">
-            <hardwareInterface>EffortJointInterface</hardwareInterface>
+      <actuator name="${prefix}_${suffix}_wheel_motor">
+        <mechanicalReduction>1</mechanicalReduction>
+      </actuator>
+      <joint name="${prefix}_${suffix}_wheel_joint">
+        <hardwareInterface>VelocityJointInterface</hardwareInterface>
       </joint>
-      <actuator name="motor_wheel_${prefix}">
-            <hardwareInterface>EffortJointInterface</hardwareInterface>
-            <mechanicalReduction>1</mechanicalReduction>
-      </actuator>
     </transmission>
-    <xacro:roller prefix="${prefix}" suffix="right_one" theta="${pi * ( 1/6)}" side="-1"/>
-    <xacro:roller prefix="${prefix}" suffix="right_two" theta="${pi * ( 2/6)}" side="-1"/>
-    <xacro:roller prefix="${prefix}" suffix="right_thr" theta="${pi * ( 3/6)}" side="-1"/>
-    <xacro:roller prefix="${prefix}" suffix="right_for" theta="${pi * ( 4/6)}" side="-1"/>
-    <xacro:roller prefix="${prefix}" suffix="right_fve" theta="${pi * ( 5/6)}" side="-1"/>
-    <xacro:roller prefix="${prefix}" suffix="right_six" theta="${pi * ( 6/6)}" side="-1"/>
-    <xacro:roller prefix="${prefix}" suffix="right_svn" theta="${pi * ( 7/6)}" side="-1"/>
-    <xacro:roller prefix="${prefix}" suffix="right_ate" theta="${pi * ( 8/6)}" side="-1"/>
-    <xacro:roller prefix="${prefix}" suffix="right_nne" theta="${pi * ( 9/6)}" side="-1"/>
-    <xacro:roller prefix="${prefix}" suffix="right_ten" theta="${pi * (10/6)}" side="-1"/>
-    <xacro:roller prefix="${prefix}" suffix="right_lvn" theta="${pi * (11/6)}" side="-1"/>
-    <xacro:roller prefix="${prefix}" suffix="right_wlv" theta="${pi * (12/6)}" side="-1"/>
-    <xacro:roller prefix="${prefix}" suffix="left_one" theta="${pi * ( 1/6) + ( pi / 12 )}" side="1"/>
-    <xacro:roller prefix="${prefix}" suffix="left_two" theta="${pi * ( 2/6) + ( pi / 12 )}" side="1"/>
-    <xacro:roller prefix="${prefix}" suffix="left_thr" theta="${pi * ( 3/6) + ( pi / 12 )}" side="1"/>
-    <xacro:roller prefix="${prefix}" suffix="left_for" theta="${pi * ( 4/6) + ( pi / 12 )}" side="1"/>
-    <xacro:roller prefix="${prefix}" suffix="left_fve" theta="${pi * ( 5/6) + ( pi / 12 )}" side="1"/>
-    <xacro:roller prefix="${prefix}" suffix="left_six" theta="${pi * ( 6/6) + ( pi / 12 )}" side="1"/>
-    <xacro:roller prefix="${prefix}" suffix="left_svn" theta="${pi * ( 7/6) + ( pi / 12 )}" side="1"/>
-    <xacro:roller prefix="${prefix}" suffix="left_ate" theta="${pi * ( 8/6) + ( pi / 12 )}" side="1"/>
-    <xacro:roller prefix="${prefix}" suffix="left_nne" theta="${pi * ( 9/6) + ( pi / 12 )}" side="1"/>
-    <xacro:roller prefix="${prefix}" suffix="left_ten" theta="${pi * (10/6) + ( pi / 12 )}" side="1"/>
-    <xacro:roller prefix="${prefix}" suffix="left_lvn" theta="${pi * (11/6) + ( pi / 12 )}" side="1"/>
-    <xacro:roller prefix="${prefix}" suffix="left_wlv" theta="${pi * (12/6) + ( pi / 12 )}" side="1"/>
-</xacro:macro>
-<xacro:wheel prefix="front_right" changeInX=" .17145" changeInY=" .10145"/>
-<xacro:wheel prefix="front_left " changeInX="-.17145" changeInY=" .10145"/>
-<xacro:wheel prefix="back_right " changeInX=" .17145" changeInY="-.10145"/>
-<xacro:wheel prefix="back_left  " changeInX="-.17145" changeInY="-.10145"/>
-<gazebo>
-  <plugin name="gazebo_ros_control" filename="libgazebo_ros_control.so">
-    <robotNamespace>/</robotNamespace>
-  </plugin>
-</gazebo>
+    <xacro:roller prefix="${prefix}_${suffix}" suffix="right_one" theta="${pi * ( 1/6)}" side="-1"/>
+    <xacro:roller prefix="${prefix}_${suffix}" suffix="right_two" theta="${pi * ( 2/6)}" side="-1"/>
+    <xacro:roller prefix="${prefix}_${suffix}" suffix="right_thr" theta="${pi * ( 3/6)}" side="-1"/>
+    <xacro:roller prefix="${prefix}_${suffix}" suffix="right_for" theta="${pi * ( 4/6)}" side="-1"/>
+    <xacro:roller prefix="${prefix}_${suffix}" suffix="right_fve" theta="${pi * ( 5/6)}" side="-1"/>
+    <xacro:roller prefix="${prefix}_${suffix}" suffix="right_six" theta="${pi * ( 6/6)}" side="-1"/>
+    <xacro:roller prefix="${prefix}_${suffix}" suffix="right_svn" theta="${pi * ( 7/6)}" side="-1"/>
+    <xacro:roller prefix="${prefix}_${suffix}" suffix="right_ate" theta="${pi * ( 8/6)}" side="-1"/>
+    <xacro:roller prefix="${prefix}_${suffix}" suffix="right_nne" theta="${pi * ( 9/6)}" side="-1"/>
+    <xacro:roller prefix="${prefix}_${suffix}" suffix="right_ten" theta="${pi * (10/6)}" side="-1"/>
+    <xacro:roller prefix="${prefix}_${suffix}" suffix="right_lvn" theta="${pi * (11/6)}" side="-1"/>
+    <xacro:roller prefix="${prefix}_${suffix}" suffix="right_wlv" theta="${pi * (12/6)}" side="-1"/>
+    <xacro:roller prefix="${prefix}_${suffix}" suffix="left_one" theta="${pi * ( 1/6) + ( pi / 12 )}" side="1"/>
+    <xacro:roller prefix="${prefix}_${suffix}" suffix="left_two" theta="${pi * ( 2/6) + ( pi / 12 )}" side="1"/>
+    <xacro:roller prefix="${prefix}_${suffix}" suffix="left_thr" theta="${pi * ( 3/6) + ( pi / 12 )}" side="1"/>
+    <xacro:roller prefix="${prefix}_${suffix}" suffix="left_for" theta="${pi * ( 4/6) + ( pi / 12 )}" side="1"/>
+    <xacro:roller prefix="${prefix}_${suffix}" suffix="left_fve" theta="${pi * ( 5/6) + ( pi / 12 )}" side="1"/>
+    <xacro:roller prefix="${prefix}_${suffix}" suffix="left_six" theta="${pi * ( 6/6) + ( pi / 12 )}" side="1"/>
+    <xacro:roller prefix="${prefix}_${suffix}" suffix="left_svn" theta="${pi * ( 7/6) + ( pi / 12 )}" side="1"/>
+    <xacro:roller prefix="${prefix}_${suffix}" suffix="left_ate" theta="${pi * ( 8/6) + ( pi / 12 )}" side="1"/>
+    <xacro:roller prefix="${prefix}_${suffix}" suffix="left_nne" theta="${pi * ( 9/6) + ( pi / 12 )}" side="1"/>
+    <xacro:roller prefix="${prefix}_${suffix}" suffix="left_ten" theta="${pi * (10/6) + ( pi / 12 )}" side="1"/>
+    <xacro:roller prefix="${prefix}_${suffix}" suffix="left_lvn" theta="${pi * (11/6) + ( pi / 12 )}" side="1"/>
+    <xacro:roller prefix="${prefix}_${suffix}" suffix="left_wlv" theta="${pi * (12/6) + ( pi / 12 )}" side="1"/>
+  </xacro:macro>
+  <xacro:wheel prefix="left" suffix="front"  reflect= "1" reflectX="-1"/>
+  <xacro:wheel prefix="left" suffix="back"   reflect="-1" reflectX="-1"/>
+  <xacro:wheel prefix="right" suffix="front" reflect= "1" reflectX= "1"/>
+  <xacro:wheel prefix="right" suffix="back"  reflect="-1" reflectX= "1"/>
+  <!-- Gazebo plugin for ROS Control -->
+  <gazebo>
+    <plugin name="gazebo_ros_control" filename="libgazebo_ros_control.so">
+      <robotNamespace>/</robotNamespace>
+    </plugin>
+  </gazebo>
 </robot>

Commit message: Update innertias

File: urdf/robot.urdf.xacro (robot description, xacro)
@@ -28,8 +28,14 @@
     <color rgba="1 1 1 1"/>
   </material>
+  <xacro:macro name="chassis_inertial" params="mass">
+    <inertial>
+      <mass value="${mass}" />
+      <inertia ixx="0.5" ixy="0.0" ixz="0.0" iyy="0.5" iyz="0.0" izz="0.3" />
+    </inertial>
+  </xacro:macro>
   <xacro:macro name="default_inertial" params="mass">
     <inertial>
       <mass value="${mass}" />
-      <inertia ixx="1.0" ixy="0.0" ixz="0.0" iyy="1.0" iyz="0.0" izz="1.0" />
+      <inertia ixx="0.00001" ixy="0.0" ixz="0.0" iyy="0.00001" iyz="0.0" izz="0.00001" />
     </inertial>
   </xacro:macro>
@@ -46,5 +52,5 @@
       </geometry>
     </collision>
-    <xacro:default_inertial mass="10"/>
+    <xacro:chassis_inertial mass="10"/>
   </link>
   <xacro:macro name="roller" params="prefix suffix theta side">
@@ -63,5 +69,5 @@
         </geometry>
       </collision>
-      <xacro:default_inertial mass="1"/>
+      <xacro:default_inertial mass="0.001"/>
     </link>
     <joint name="${prefix}_${suffix}_roller_joint" type="continuous">
@@ -107,5 +113,5 @@
         </geometry>
       </collision>
-      <xacro:default_inertial mass="1"/>
+      <xacro:default_inertial mass="0.001"/>
     </link>
     <joint name="${prefix}_${suffix}_wheel_joint" type="continuous">

Commit message: Clean up

File: urdf/robot.urdf.xacro (robot description, xacro)
@@ -31,5 +31,5 @@
     <inertial>
       <mass value="${mass}" />
-      <inertia ixx="0.5" ixy="0.0" ixz="0.0" iyy="0.5" iyz="0.0" izz="0.3" />
+      <inertia ixx="0.5" ixy="0.0" ixz="0.0" iyy="0.3" iyz="0.0" izz="0.5" />
     </inertial>
   </xacro:macro>
@@ -72,5 +72,5 @@
     </link>
     <joint name="${prefix}_${suffix}_roller_joint" type="continuous">
-      <axis xyz="0 1 0" rpy="0 0 0" />
+      <axis xyz="1 0 0" />
       <parent link="${prefix}_wheel"/>
       <child link="${prefix}_${suffix}_roller"/>
@@ -79,11 +79,4 @@
     <!-- This block provides the simulator (Gazebo) with information on a few additional
     physical properties. See http://gazebosim.org/tutorials/?tut=ros_urdf for more-->
-    <gazebo reference="${prefix}_${suffix}_roller">
-      <mu1 value="200.0"/>
-      <mu2 value="100.0"/>
-      <kp value="10000000.0" />
-      <kd value="1.0" />
-      <material>Gazebo/Grey</material>
-    </gazebo>
     <!-- This block connects the wheel joint to an actuator (motor), which informs both
     simulation and visualization of the robot -->
@@ -116,5 +109,5 @@
     </link>
     <joint name="${prefix}_${suffix}_wheel_joint" type="continuous">
-      <axis xyz="0 1 0" rpy="0 0 0" />
+      <axis xyz="0 1 0" />
       <parent link="base_link"/>
       <child link="${prefix}_${suffix}_wheel"/>
