Commit message: load faster

File: urdf/robot.urdf.xacro (robot description, xacro)
@@ -19,4 +19,5 @@
     <xacro:property name="roller_side_length" value="0.0088"/>
     <xacro:property name="roller_radius" value=".0475"/>
+    <xacro:property name="default_start" value="0 0 0"/>
     <material name="blue">
         <color rgba="0 0 0.8 1"/>
@@ -42,5 +43,5 @@
     <link name="base_link">
         <visual>
-            <origin xyz="0 0 0" rpy="0 0 0" />
+            <origin xyz="${default_start}" rpy="0 0 0" />
             <geometry>
                 <cylinder radius="${width}" length="${bodylen}"/>
@@ -49,5 +50,5 @@
         </visual>
         <collision>
-            <origin xyz="0 0 0" rpy="0 0 0" />
+            <origin xyz="${default_start}" rpy="0 0 0" />
             <geometry>
                 <cylinder radius="${width}" length="${bodylen}"/>
@@ -59,5 +60,5 @@
         <link name="${prefix}_${suffix}_roller">
             <visual>
-                <origin xyz="0 0 0" rpy="0 ${pi/2} 0" />
+                <origin xyz="${default_start}" rpy="0 ${pi/2} 0" />
                 <geometry>
                     <cylinder radius="${roller_diameter}" length="${roller_width}"/>
@@ -66,5 +67,5 @@
             </visual>
             <collision>
-                <origin xyz="0 0 0" rpy="0 ${pi/2} 0" />
+                <origin xyz="${default_start}" rpy="0 ${pi/2} 0" />
                 <geometry>
                     <cylinder radius="${roller_diameter}" length="${roller_width}"/>
@@ -95,5 +96,5 @@
         <link name="${prefix}_${suffix}_wheel">
             <visual>
-                <origin xyz="0 0 0" rpy="${pi/2} 0 0" />
+                <origin xyz="${default_start}" rpy="${pi/2} 0 0" />
                 <geometry>
                     <cylinder radius="${wheeldiam/2}" length="${wheel_width}"/>
@@ -102,5 +103,5 @@
             </visual>
             <collision>
-                <origin xyz="0 0 0" rpy="${pi/2} 0 0" />
+                <origin xyz="${default_start}" rpy="${pi/2} 0 0" />
                 <geometry>
                     <cylinder radius="${wheeldiam/2}" length="${wheel_width}"/>
@@ -164,10 +165,9 @@
     <xacro:wheel prefix="right" suffix="front" reflect= "1" reflectX= "1"/>
     <xacro:wheel prefix="right" suffix="back"  reflect="-1" reflectX= "1"/>
-    <link name="dummy">
-   </link>
-     <joint name="dummy_joint" type="fixed">
-     <parent link="dummy"/>
-     <child link="base_link"/>
-   </joint>
+    <link name="dummy"/>
+    <joint name="dummy_joint" type="fixed">
+        <parent link="dummy"/>
+        <child link="base_link"/>
+    </joint>
     <!-- Gazebo plugin for ROS Control -->
     <gazebo>

Commit message: changed place to start

File: urdf/robot.urdf.xacro (robot description, xacro)
@@ -19,5 +19,4 @@
     <xacro:property name="roller_side_length" value="0.0088"/>
     <xacro:property name="roller_radius" value=".0475"/>
-    <xacro:property name="default_start" value="0 0 0"/>
     <material name="blue">
         <color rgba="0 0 0.8 1"/>
@@ -43,5 +42,5 @@
     <link name="base_link">
         <visual>
-            <origin xyz="${default_start}" rpy="0 0 0" />
+            <origin xyz="0 0 0" rpy="0 0 0" />
             <geometry>
                 <cylinder radius="${width}" length="${bodylen}"/>
@@ -50,5 +49,5 @@
         </visual>
         <collision>
-            <origin xyz="${default_start}" rpy="0 0 0" />
+            <origin xyz="0 0 0" rpy="0 0 0" />
             <geometry>
                 <cylinder radius="${width}" length="${bodylen}"/>
@@ -60,5 +59,5 @@
         <link name="${prefix}_${suffix}_roller">
             <visual>
-                <origin xyz="${default_start}" rpy="0 ${pi/2} 0" />
+                <origin xyz="0 0 0" rpy="0 ${pi/2} 0" />
                 <geometry>
                     <cylinder radius="${roller_diameter}" length="${roller_width}"/>
@@ -67,5 +66,5 @@
             </visual>
             <collision>
-                <origin xyz="${default_start}" rpy="0 ${pi/2} 0" />
+                <origin xyz="0 0 0" rpy="0 ${pi/2} 0" />
                 <geometry>
                     <cylinder radius="${roller_diameter}" length="${roller_width}"/>
@@ -96,5 +95,5 @@
         <link name="${prefix}_${suffix}_wheel">
             <visual>
-                <origin xyz="${default_start}" rpy="${pi/2} 0 0" />
+                <origin xyz="0 0 0" rpy="${pi/2} 0 0" />
                 <geometry>
                     <cylinder radius="${wheeldiam/2}" length="${wheel_width}"/>
@@ -103,5 +102,5 @@
             </visual>
             <collision>
-                <origin xyz="${default_start}" rpy="${pi/2} 0 0" />
+                <origin xyz="0 0 0" rpy="${pi/2} 0 0" />
                 <geometry>
                     <cylinder radius="${wheeldiam/2}" length="${wheel_width}"/>
@@ -165,9 +164,9 @@
     <xacro:wheel prefix="right" suffix="front" reflect= "1" reflectX= "1"/>
     <xacro:wheel prefix="right" suffix="back"  reflect="-1" reflectX= "1"/>
-    <link name="dummy"/>
-    <joint name="dummy_joint" type="fixed">
-        <parent link="dummy"/>
-        <child link="base_link"/>
-    </joint>
+    <link name="dummy"></link>
+     <joint name="dummy_joint" type="fixed">
+     <parent link="dummy"/>
+     <child link="base_link"/>
+   </joint>
     <!-- Gazebo plugin for ROS Control -->
     <gazebo>

Commit message: added camera to robot | still need to figure out how to publish the camera topic... it works with depth camera test

File: urdf/robot.urdf.xacro (robot description, xacro)
@@ -165,8 +165,112 @@
     <xacro:wheel prefix="right" suffix="back"  reflect="-1" reflectX= "1"/>
     <link name="dummy"></link>
-     <joint name="dummy_joint" type="fixed">
-     <parent link="dummy"/>
-     <child link="base_link"/>
-   </joint>
+    <joint name="dummy_joint" type="fixed">
+        <parent link="dummy"/>
+        <child link="base_link"/>
+    </joint>
+    <link name="camera_link">
+      <pose frame=''>0.056797 -0.011425 0.036 0 -0 0</pose>
+        <!--<inertial>
+          <mass>0.1</mass>
+        </inertial>-->
+        <collision name="collision">
+            <origin rpy="0 0 0" xyz="0 0 0"/>
+            <geometry>
+                <mesh filename="package://gazeboSimulation/models/kinect/meshes/kinect.dae"/>
+            </geometry>
+        </collision>
+        <visual name="visual">
+            <origin rpy="0 0 0" xyz="0 0 0"/>
+            <geometry>
+                <mesh filename="package://gazeboSimulation/models/kinect/meshes/kinect.dae"/>
+            </geometry>
+        </visual>
+          <!-- camera -->
+  <gazebo reference="camera_link">
+    <sensor type="camera" name="camera1">
+      <update_rate>30.0</update_rate>
+      <camera name="head">
+        <horizontal_fov>1.3962634</horizontal_fov>
+        <image>
+          <width>800</width>
+          <height>800</height>
+          <format>R8G8B8</format>
+        </image>
+        <clip>
+          <near>0.02</near>
+          <far>300</far>
+        </clip>
+        <noise>
+          <type>gaussian</type>
+          <!-- Noise is sampled independently per pixel on each frame.
+               That pixel's noise value is added to each of its color
+               channels, which at that point lie in the range [0,1]. -->
+          <mean>0.0</mean>
+          <stddev>0.007</stddev>
+        </noise>
+      </camera>
+      <plugin name="camera_controller" filename="libgazebo_ros_camera.so">
+        <alwaysOn>true</alwaysOn>
+        <updateRate>0.0</updateRate>
+        <cameraName>rrbot/camera1</cameraName>
+        <imageTopicName>image_raw</imageTopicName>
+        <cameraInfoTopicName>camera_info</cameraInfoTopicName>
+        <frameName>camera_link</frameName>
+        <hackBaseline>0.07</hackBaseline>
+        <distortionK1>0.0</distortionK1>
+        <distortionK2>0.0</distortionK2>
+        <distortionK3>0.0</distortionK3>
+        <distortionT1>0.0</distortionT1>
+        <distortionT2>0.0</distortionT2>
+      </plugin>
+    </sensor>
+  </gazebo><!--
+        <gazebo reference="camera_link">
+            <sensor name="camera" type="depth">
+                <update_rate>20</update_rate>
+                <camera>
+                    <horizontal_fov>1.047198</horizontal_fov>
+                    <image>
+                        <width>640</width>
+                        <height>480</height>
+                        <format>R8G8B8</format>
+                    </image>
+                    <clip>
+                        <near>0.05</near>
+                        <far>3</far>
+                    </clip>
+                </camera>
+                <plugin name="camera_plugin" filename="libgazebo_ros_openni_kinect.so">
+                    <baseline>0.2</baseline>
+                    <alwaysOn>true</alwaysOn>
+                    <updateRate>0.0</updateRate>
+                    <cameraName>camera_ir</cameraName>
+                    <imageTopicName>/camera/color/image_raw</imageTopicName>
+                    <cameraInfoTopicName>/camera/color/camera_info</cameraInfoTopicName>
+                    <depthImageTopicName>/camera/depth/image_raw</depthImageTopicName>
+                    <depthImageCameraInfoTopicName>/camera/depth/camera_info</depthImageCameraInfoTopicName>
+                    <pointCloudTopicName>/camera/depth/points</pointCloudTopicName>
+                    <frameName>camera_link</frameName>
+                    <pointCloudCutoff>0.5</pointCloudCutoff>
+                    <pointCloudCutoffMax>3.0</pointCloudCutoffMax>
+                    <distortionK1>0</distortionK1>
+                    <distortionK2>0</distortionK2>
+                    <distortionK3>0</distortionK3>
+                    <distortionT1>0</distortionT1>
+                    <distortionT2>0</distortionT2>
+                    <CxPrime>0</CxPrime>
+                    <Cx>0</Cx>
+                    <Cy>0</Cy>
+                    <focalLength>0</focalLength>
+                    <hackBaseline>0</hackBaseline>
+                </plugin>
+            </sensor>
+        </gazebo>-->
+    </link>
+    <joint name="camera_joint" type="fixed">
+        <child link="camera_link"/>
+        <parent link="base_link"/>
+        <origin rpy="0 0 0" xyz="0 0 .15"/>
+    </joint>
     <!-- Gazebo plugin for ROS Control -->
     <gazebo>
@@ -184,30 +288,4 @@
           <rpyOffsets>0 0 0</rpyOffsets>
         </plugin>
-        <plugin name="camera_plugin" filename="libgazebo_ros_openni_kinect.so">
-          <baseline>0.2</baseline>
-          <alwaysOn>true</alwaysOn>
-          <!-- Keep this zero, update_rate in the parent <sensor> tag
-            will control the frame rate. -->
-          <updateRate>0.0</updateRate>
-          <cameraName>camera_ir</cameraName>
-          <imageTopicName>/camera/color/image_raw</imageTopicName>
-          <cameraInfoTopicName>/camera/color/camera_info</cameraInfoTopicName>
-          <depthImageTopicName>/camera/depth/image_raw</depthImageTopicName>
-          <depthImageCameraInfoTopicName>/camera/depth/camera_info</depthImageCameraInfoTopicName>
-          <pointCloudTopicName>/camera/depth/points</pointCloudTopicName>
-          <frameName>camera_link</frameName>
-          <pointCloudCutoff>0.5</pointCloudCutoff>
-          <pointCloudCutoffMax>3.0</pointCloudCutoffMax>
-          <distortionK1>0</distortionK1>
-          <distortionK2>0</distortionK2>
-          <distortionK3>0</distortionK3>
-          <distortionT1>0</distortionT1>
-          <distortionT2>0</distortionT2>
-          <CxPrime>0</CxPrime>
-          <Cx>0</Cx>
-          <Cy>0</Cy>
-          <focalLength>0</focalLength>
-          <hackBaseline>0</hackBaseline>
-        </plugin>
     </gazebo>
 </robot>
