Commit message: Bug fixes. odom works correctly,  kinect works

File: urdf/camera.urdf.xacro (robot description, xacro)
@@ -2,15 +2,16 @@
 <robot name="chassis" xmlns:xacro="http://ros.org/wiki/xacro">
     <xacro:property name="M_PI" value="3.1415926535897931" />
-    <link name="camera_link">
+    <xacro:macro name="kinect" params="prefix origin_link xyz rpy">
+    <link name="${prefix}_camera_link">
       <visual>
-        <origin xyz="0 0 0" rpy="0 1.5708 1.5708"/>
+        <origin xyz="0 0 0" rpy="0 0 0"/>
         <geometry>
-          <box size="0.5 0.1 0.03"/>
+          <box size="0.01 0.05 0.03"/>
         </geometry>
       </visual>
       <collision>
-        <origin xyz="0 0 0" rpy="0 1.5708 1.5708"/>
+        <origin xyz="0 0 0" rpy="0 0 0"/>
         <geometry>
-          <box size="0.5 0.1 0.03"/>
+          <box size="0.01 0.05 0.03"/>
         </geometry>
       </collision>
@@ -23,10 +24,21 @@
       </inertial>
     </link>
+    <joint name="${prefix}_camera_joint" type="fixed">
+        <parent link="${origin_link}"/>
+        <child link="${prefix}_camera_link"/>
+        <origin rpy="${rpy}" xyz="${xyz}"/>
+    </joint>
+    <link name="${prefix}_lens_link"></link>
+    <joint name="${prefix}_lens_joint" type="fixed">
+        <parent link="${prefix}_camera_link"/>
+        <child link="${prefix}_lens_link"/>
+        <origin xyz="0 0 0" rpy="-1.57 0 -1.57"/>
+    </joint>
         <!-- camera -->
-    <gazebo reference="camera_link">
+    <gazebo reference="${prefix}_camera_link">
       <sensor type="depth" name="camera_link_sensor">
         <!-- offset between camera_link and camera_depth_optical_link -->
         <!-- additional mm offsets added through inspection -->
-        <pose>-0.001 -0.045 0.001 -0.000 0 0</pose>
+        <pose>-0.001 -0.045 0.001 -0.000 0 1.57</pose>
         <always_on>true</always_on>
         <update_rate>15.0</update_rate>
@@ -46,11 +58,11 @@
           <alwaysOn>true</alwaysOn>
           <updateRate>15.0</updateRate>
-          <cameraName>camera</cameraName>
-          <frameName>camera_link</frameName>
-          <imageTopicName>/camera/rgb/image_rect_color</imageTopicName>
-          <cameraInfoTopicName>/camera/rgb/camera_info</cameraInfoTopicName>
-          <depthImageTopicName>/camera/depth_registered/image_raw</depthImageTopicName>
-          <depthImageCameraInfoTopicName>/camera/depth_registered/camera_info</depthImageCameraInfoTopicName>
-          <pointCloudTopicName>/camera/depth/points</pointCloudTopicName>
+          <cameraName>${prefix}_camera</cameraName>
+          <frameName>GT/${prefix}_lens_link</frameName>
+          <imageTopicName>${prefix}_camera/rgb/image_rect_color</imageTopicName>
+          <cameraInfoTopicName>${prefix}_camera/rgb/camera_info</cameraInfoTopicName>
+          <depthImageTopicName>${prefix}_camera/depth_registered/image_raw</depthImageTopicName>
+          <depthImageCameraInfoTopicName>${prefix}_camera/depth_registered/camera_info</depthImageCameraInfoTopicName>
+          <pointCloudTopicName>${prefix}_camera/depth/points</pointCloudTopicName>
           <pointCloudCutoff>0.5</pointCloudCutoff>
           <distortionK1>0.00000001</distortionK1>
@@ -62,3 +74,4 @@
       </sensor>
     </gazebo>
+    </xacro:macro>
 </robot>

File: urdf/chassis.urdf.xacro (robot description, xacro)
@@ -160,8 +160,8 @@
         <xacro:roller prefix="${prefix}_${suffix}" suffix="left_wlv" theta="${pi * (12/6) + ( pi / 12 )}" side="1"/>
     </xacro:macro>
-    <xacro:wheel prefix="left" suffix="front"  reflect= "1" reflectX="-1"/>
-    <xacro:wheel prefix="left" suffix="back"   reflect="-1" reflectX="-1"/>
-    <xacro:wheel prefix="right" suffix="front" reflect= "1" reflectX= "1"/>
-    <xacro:wheel prefix="right" suffix="back"  reflect="-1" reflectX= "1"/>
+    <xacro:wheel prefix="left" suffix="front"  reflect= "1" reflectX="1"/>
+    <xacro:wheel prefix="left" suffix="back"   reflect="-1" reflectX="1"/>
+    <xacro:wheel prefix="right" suffix="front" reflect= "1" reflectX= "-1"/>
+    <xacro:wheel prefix="right" suffix="back"  reflect="-1" reflectX= "-1"/>
     <!-- Gazebo plugin for ROS Control -->
     <gazebo>

File: urdf/robot.urdf.xacro (robot description, xacro)
@@ -2,14 +2,11 @@
 <robot name="roscontrol" xmlns:xacro="http://ros.org/wiki/xacro">
     <link name="base_link"></link>
-    <xacro:include filename="chassis.urdf.xacro" ns="chassis"/>
+    <xacro:include filename="chassis.urdf.xacro"/>
     <joint name="chassis_joint" type="fixed">
         <parent link="base_link"/>
         <child link="chassis_link"/>
     </joint>
-    <xacro:include filename="camera.urdf.xacro" ns="camera"/>
-    <joint name="camera_joint" type="fixed">
-        <parent link="base_link"/>
-        <child link="camera_link"/>
-        <origin rpy="0 0 0" xyz="0 0 .1"/>
-    </joint><!---->
+    <xacro:include filename="camera.urdf.xacro"/>
+    <xacro:kinect prefix="front" origin_link="base_link" xyz="0.1 0 0.1" rpy="0 0 0"/>
+    <xacro:kinect prefix="back" origin_link="base_link" xyz="-0.1 0 0.1" rpy="0 0 3.14"/>
 </robot>

Commit message: no

File: urdf/camera.urdf.xacro (robot description, xacro)
@@ -4,13 +4,13 @@
     <link name="camera_link">
       <visual>
-        <origin xyz="0 0 0" rpy="0 1.5708 1.5708"/>
+        <origin xyz="0 0 0" rpy="1.5707635 0 0"/>
         <geometry>
-          <box size="0.5 0.1 0.03"/>
+          <box size="0.05 0.1 0.03"/>
         </geometry>
       </visual>
       <collision>
-        <origin xyz="0 0 0" rpy="0 1.5708 1.5708"/>
+        <origin xyz="0 0 0" rpy="1.5707635 0 0"/>
         <geometry>
-          <box size="0.5 0.1 0.03"/>
+          <box size="0.05 0.1 0.03"/>
         </geometry>
       </collision>
@@ -23,5 +23,5 @@
       </inertial>
     </link>
-        <!-- camera -->
+    <!-- camera -->
     <gazebo reference="camera_link">
       <sensor type="depth" name="camera_link_sensor">

File: urdf/depth_camera_test.urdf.xacro (robot description, xacro)
@@ -1,64 +1,10 @@
 <?xml version="1.0"?>
-<robot xmlns:xacro="http://www.ros.org/wiki/xacro" name="depth_camera_test_urdf">
-    <pose>0 0 0 0 0 0</pose>
-    <link name="camera_link">
-        <!--<inertial>
-          <mass>0.1</mass>
-        </inertial>-->
-        <collision name="collision">
-            <origin rpy="0 0 0" xyz="0 0 0"/>
-            <geometry>
-                <mesh filename="package://gazeboSimulation/models/kinect/meshes/kinect.dae"/>
-            </geometry>
-        </collision>
-        <visual name="visual">
-            <origin rpy="0 0 0" xyz="0 0 0"/>
-            <geometry>
-                <mesh filename="package://gazeboSimulation/models/kinect/meshes/kinect.dae"/>
-            </geometry>
-        </visual>
-        <gazebo>
-            <sensor name="camera" type="depth">
-                <update_rate>20</update_rate>
-                <camera>
-                    <horizontal_fov>1.047198</horizontal_fov>
-                    <image>
-                        <width>640</width>
-                        <height>480</height>
-                        <format>R8G8B8</format>
-                    </image>
-                    <clip>
-                        <near>0.05</near>
-                        <far>3</far>
-                    </clip>
-                </camera>
-                <plugin name="camera_plugin" filename="libgazebo_ros_openni_kinect.so">
-                    <baseline>0.2</baseline>
-                    <alwaysOn>true</alwaysOn>
-                    <!-- Keep this zero, update_rate in the parent <sensor> tag
-                      will control the frame rate. -->
-                    <updateRate>0.0</updateRate>
-                    <cameraName>camera_ir</cameraName>
-                    <imageTopicName>/camera/color/image_raw</imageTopicName>
-                    <cameraInfoTopicName>/camera/color/camera_info</cameraInfoTopicName>
-                    <depthImageTopicName>/camera/depth/image_raw</depthImageTopicName>
-                    <depthImageCameraInfoTopicName>/camera/depth/camera_info</depthImageCameraInfoTopicName>
-                    <pointCloudTopicName>/camera/depth/points</pointCloudTopicName>
-                    <frameName>camera_link</frameName>
-                    <pointCloudCutoff>0.5</pointCloudCutoff>
-                    <pointCloudCutoffMax>3.0</pointCloudCutoffMax>
-                    <distortionK1>0</distortionK1>
-                    <distortionK2>0</distortionK2>
-                    <distortionK3>0</distortionK3>
-                    <distortionT1>0</distortionT1>
-                    <distortionT2>0</distortionT2>
-                    <CxPrime>0</CxPrime>
-                    <Cx>0</Cx>
-                    <Cy>0</Cy>
-                    <focalLength>0</focalLength>
-                    <hackBaseline>0</hackBaseline>
-                </plugin>
-            </sensor>
-        </gazebo>
-    </link>
+<robot name="roscontrol" xmlns:xacro="http://ros.org/wiki/xacro">
+    <link name="base_link"></link>
+    <xacro:include filename="camera.urdf.xacro" ns="camera"/>
+    <joint name="camera_joint" type="fixed">
+        <parent link="base_link"/>
+        <child link="camera_link"/>
+        <origin xyz="0 0 .1" rpy="0 0 0" />
+    </joint><!---->
 </robot>

File: urdf/robot.urdf.xacro (robot description, xacro)
@@ -11,5 +11,5 @@
         <parent link="base_link"/>
         <child link="camera_link"/>
-        <origin rpy="0 0 0" xyz="0 0 .1"/>
+        <origin xyz="0 0 .1" rpy="0 0 0" />
     </joint><!---->
 </robot>

Commit message: fixed master being destroyed

File: urdf/camera.urdf.xacro (robot description, xacro)
@@ -5,15 +5,4 @@
     <link name="${prefix}_camera_link">
       <visual>
-<<<<<<< HEAD
-        <origin xyz="0 0 0" rpy="1.5707635 0 0"/>
-        <geometry>
-          <box size="0.05 0.1 0.03"/>
-        </geometry>
-      </visual>
-      <collision>
-        <origin xyz="0 0 0" rpy="1.5707635 0 0"/>
-        <geometry>
-          <box size="0.05 0.1 0.03"/>
-=======
         <origin xyz="0 0 0" rpy="0 0 0"/>
         <geometry>
@@ -25,5 +14,4 @@
         <geometry>
           <box size="0.01 0.05 0.03"/>
->>>>>>> master
         </geometry>
       </collision>
@@ -36,8 +24,4 @@
       </inertial>
     </link>
-<<<<<<< HEAD
-    <!-- camera -->
-    <gazebo reference="camera_link">
-=======
     <joint name="${prefix}_camera_joint" type="fixed">
         <parent link="${origin_link}"/>
@@ -53,5 +37,4 @@
         <!-- camera -->
     <gazebo reference="${prefix}_camera_link">
->>>>>>> master
       <sensor type="depth" name="camera_link_sensor">
         <!-- offset between camera_link and camera_depth_optical_link -->

File: urdf/robot.urdf.xacro (robot description, xacro)
@@ -7,15 +7,6 @@
         <child link="chassis_link"/>
     </joint>
-<<<<<<< HEAD
-    <xacro:include filename="camera.urdf.xacro" ns="camera"/>
-    <joint name="camera_joint" type="fixed">
-        <parent link="base_link"/>
-        <child link="camera_link"/>
-        <origin xyz="0 0 .1" rpy="0 0 0" />
-    </joint><!---->
-=======
     <xacro:include filename="camera.urdf.xacro"/>
     <xacro:kinect prefix="front" origin_link="base_link" xyz="0.1 0 0.1" rpy="0 0 0"/>
     <xacro:kinect prefix="back" origin_link="base_link" xyz="-0.1 0 0.1" rpy="0 0 3.14"/>
->>>>>>> master
 </robot>

Commit message: balls can now be put in robot if in radius

File: urdf/camera.urdf.xacro (robot description, xacro)
@@ -7,5 +7,5 @@
         <origin xyz="0 0 0" rpy="0 0 0"/>
         <geometry>
-          <box size="0.01 0.05 0.03"/>
+          <box size="0.01 0.05 0.3"/>
         </geometry>
       </visual>
@@ -13,5 +13,5 @@
         <origin xyz="0 0 0" rpy="0 0 0"/>
         <geometry>
-          <box size="0.01 0.05 0.03"/>
+          <box size="0.01 0.05 0.3"/>
         </geometry>
       </collision>
