Commit message: the "full" robot, still needs some tuning but I need sleep, cuz its like 4:52

File: urdf/FlyWheel.urdf.xacro (robot description, xacro)
@@ -164,17 +164,18 @@
     </link>
 </xacro:macro>-->
-<xacro:macro name="intake" params="prefix suffix reflect reflectX">
+<xacro:macro name="intake" params="prefix suffix reflect reflectX z_val">
     <link name="${prefix}_${suffix}_intake">
         <visual>
             <origin xyz="0 0 0" rpy="0 0 0" />
             <geometry>
-                <box size="0.082 0.082 0.002"/>
-            </geometry>
-            <material name="black"/>
-        </visual>
-        <collision>
-            <origin xyz="0 0 0" rpy="0 0 0" />
-            <geometry>
-                <box size="0.082 0.082 0.002"/>
+                <cylinder radius="0.04" length=".05"/>
+                <!--<box size="0.082 0.082 0.05"/>-->
+            </geometry>
+            <material name="black"/>
+        </visual>
+        <collision>
+            <origin xyz="0 0 0" rpy="0 ${-pi/6} 0" />
+            <geometry>
+                <cylinder radius="0.04" length=".05"/>
             </geometry>
         </collision>
@@ -185,5 +186,5 @@
         <parent link="chassis_link"/>
         <child link="${prefix}_${suffix}_intake"/>
-        <origin xyz="${.2*reflect} ${.1*reflectX} 0.025" rpy="0 0 0"/>
+        <origin xyz="${.2*reflect} ${.1*reflectX} ${z_val}" rpy="0 ${-pi/6} 0"/>
     </joint>
     <!-- This block provides the simulator (Gazebo) with information on a few additional
@@ -208,4 +209,49 @@
     </transmission>
 </xacro:macro>
+<xacro:macro name="indexer" params="prefix radius z_val x_val">
+    <link name="${prefix}_indexer">
+        <visual>
+            <origin xyz="0 0 0" rpy="${pi/2} 0 0" />
+            <geometry>
+                <cylinder radius="${radius}" length=".09"/>
+                <!--<box size="${radius*2} ${radius*2} .05"/>-->
+            </geometry>
+            <material name="black"/>
+        </visual>
+        <collision>
+            <origin xyz="0 0 0" rpy="${pi/2} 0 0" />
+            <geometry>
+                <cylinder radius="${radius}" length=".09"/>
+            </geometry>
+        </collision>
+        <xacro:roller_inertial mass="0.001"/>
+    </link>
+    <joint name="${prefix}_indexer_joint" type="continuous">
+        <axis xyz="0 1 0" />
+        <parent link="chassis_link"/>
+        <child link="${prefix}_indexer"/>
+        <origin xyz="${x_val} 0 ${z_val}" rpy="0 0 0"/>
+    </joint>
+    <!-- This block provides the simulator (Gazebo) with information on a few additional
+    physical properties. See http://gazebosim.org/tutorials/?tut=ros_urdf for more-->
+    <gazebo reference="${prefix}_indexer">
+        <mu1 value="200.0"/>
+        <mu2 value="100.0"/>
+        <kp value="10000000.0" />
+        <kd value="1.0" />
+        <material>Gazebo/Green</material>
+    </gazebo>
+    <!-- This block connects the wheel joint to an actuator (motor), which informs both
+    simulation and visualization of the robot -->
+    <transmission name="${prefix}_indexer_trans">
+        <type>transmission_interface/SimpleTransmission</type>
+        <actuator name="${prefix}_indexer_motor">
+            <mechanicalReduction>1</mechanicalReduction>
+        </actuator>
+        <joint name="${prefix}_indexer_joint">
+            <hardwareInterface>VelocityJointInterface</hardwareInterface>
+        </joint>
+    </transmission>
+</xacro:macro>
 <!--          Well this is the robot          -->
 <link name="chassis_link">
@@ -213,5 +259,5 @@
     <origin xyz="0 0 0.1177" rpy="0 0 0" />
     <geometry>
-      <mesh filename="package://gazeboSimulation/models/change_up_cad/FlyWheel/Collision/CFrame.dae"/>
+      <mesh filename="package://gazeboSimulation/models/change_up_cad/FlyWheel/Visual/Frame.dae"/>
     </geometry>
   </visual>
@@ -228,6 +274,10 @@
 <xacro:wheel prefix="right" suffix="front" reflect= "1" reflectX= "-1"/>
 <xacro:wheel prefix="right" suffix="back"  reflect="-1" reflectX= "-1"/>
-<xacro:intake prefix="right" suffix="front"  reflect="-1" reflectX= "1"/>
-<xacro:intake prefix="left" suffix="front"  reflect="-1" reflectX= "-1"/>
+<xacro:intake prefix="right" suffix="front"  reflect="-1" reflectX= "1" z_val="0.05"/>
+<xacro:intake prefix="left" suffix="front"  reflect="-1" reflectX= "-1" z_val="0.05"/>
+<xacro:intake prefix="right" suffix="back"  reflect="0" reflectX= "1" z_val="0.160"/>
+<xacro:intake prefix="left" suffix="back"  reflect="0" reflectX= "-1" z_val="0.160"/>
+<xacro:indexer prefix="top" radius=".06" z_val=".35" x_val="-.07"/>
+<xacro:indexer prefix="bottom" radius=".04" z_val=".25" x_val="-.05"/>
 <!-- Gazebo plugin for ROS Control -->
 <gazebo>

File: urdf/robot.urdf.xacro (robot description, xacro)
@@ -7,9 +7,9 @@
         <child link="chassis_link"/>
     </joint>
-    <!--<xacro:include filename="depth_camera.urdf.xacro"/>
-    <xacro:kinect prefix="front" origin_link="base_link" xyz="0.1 0 0.1" rpy="0 0 0"/>
-    <xacro:kinect prefix="back" origin_link="base_link" xyz="-0.1 0 0.1" rpy="0 0 3.14"/>
+    <xacro:include filename="depth_camera.urdf.xacro"/>
+    <xacro:kinect prefix="front" origin_link="base_link" xyz="0.15 0 0.25" rpy="0 0 0"/>
+    <xacro:kinect prefix="back" origin_link="base_link" xyz="-0.15 0 0.25" rpy="0 0 3.14"/>
     <xacro:include filename="wide_camera.urdf.xacro"/>
-    <xacro:wide prefix="left" origin_link="base_link" xyz="0 -0.1 0.5" rpy="0 1.57 1.57"/>
-    <xacro:wide prefix="right" origin_link="base_link" xyz="0 0.1 0.5" rpy="1.57 1.57 0"/>-->
+    <xacro:wide prefix="left" origin_link="base_link" xyz="0 -0.15 0.1" rpy="0 1.57 1.57"/>
+    <xacro:wide prefix="right" origin_link="base_link" xyz="0 0.15 0.1" rpy="1.57 1.57 0"/>
 </robot>
