Commit message: pre-save to set up camera blob detector.

File: urdf/depth_camera.urdf.xacro (robot description, xacro)
@@ -2,76 +2,76 @@
 <robot name="chassis" xmlns:xacro="http://ros.org/wiki/xacro">
     <xacro:property name="M_PI" value="3.1415926535897931" />
-    <xacro:macro name="kinect" params="prefix origin_link xyz rpy">
-    <link name="${prefix}_camera_link">
-      <visual>
-        <origin xyz="0 0 0" rpy="0 0 0"/>
-        <geometry>
-          <box size="0.01 0.05 0.03"/>
-        </geometry>
-      </visual>
-      <collision>
-        <origin xyz="0 0 0" rpy="0 0 0"/>
-        <geometry>
-          <box size="0.01 0.05 0.03"/>
-        </geometry>
-      </collision>
-      <inertial>
-        <mass value="0.300" />
-        <inertia
-          ixx="0.001" ixy="0" ixz="0"
-          iyy="0.001" iyz="0"
-          izz="0.01" />
-      </inertial>
-    </link>
-    <joint name="${prefix}_camera_joint" type="fixed">
-        <parent link="${origin_link}"/>
-        <child link="${prefix}_camera_link"/>
-        <origin rpy="${rpy}" xyz="${xyz}"/>
-    </joint>
-    <link name="${prefix}_lens_link"></link>
-    <joint name="${prefix}_lens_joint" type="fixed">
-        <parent link="${prefix}_camera_link"/>
-        <child link="${prefix}_lens_link"/>
-        <origin xyz="0 0 0" rpy="-1.57 0 -1.57"/>
-    </joint>
-        <!-- camera -->
-    <gazebo reference="${prefix}_camera_link">
-      <sensor type="depth" name="camera_link_sensor">
-        <!-- offset between camera_link and camera_depth_optical_link -->
-        <!-- additional mm offsets added through inspection -->
-        <pose>-0.001 -0.045 0.001 -0.000 0 1.57</pose>
-        <always_on>true</always_on>
-        <update_rate>15.0</update_rate>
-        <camera>
-          <horizontal_fov>${57.0*M_PI/180.0}</horizontal_fov>
-          <image>
-            <format>R8G8B8</format>
-            <width>640</width>
-            <height>480</height>
-          </image>
-          <clip>
-            <near>0.01</near>
-            <far>5</far>
-          </clip>
-        </camera>
-        <plugin name="kinect_camera" filename="libgazebo_ros_openni_kinect.so">
-          <alwaysOn>true</alwaysOn>
-          <updateRate>15.0</updateRate>
-          <cameraName>${prefix}_camera</cameraName>
-          <frameName>GT/${prefix}_lens_link</frameName>
-          <imageTopicName>${prefix}_camera/rgb/image_rect_color</imageTopicName>
-          <cameraInfoTopicName>${prefix}_camera/rgb/camera_info</cameraInfoTopicName>
-          <depthImageTopicName>${prefix}_camera/depth_registered/image_raw</depthImageTopicName>
-          <depthImageCameraInfoTopicName>${prefix}_camera/depth_registered/camera_info</depthImageCameraInfoTopicName>
-          <pointCloudTopicName>${prefix}_camera/depth/points</pointCloudTopicName>
-          <pointCloudCutoff>0.5</pointCloudCutoff>
-          <distortionK1>0.00000001</distortionK1>
-          <distortionK2>0.00000001</distortionK2>
-          <distortionK3>0.00000001</distortionK3>
-          <distortionT1>0.00000001</distortionT1>
-          <distortionT2>0.00000001</distortionT2>
-        </plugin>
-      </sensor>
-    </gazebo>
+      <xacro:macro name="kinect" params="prefix origin_link xyz rpy">
+      <link name="${prefix}_camera_link">
+        <visual>
+          <origin xyz="0 0 0" rpy="0 0 0"/>
+          <geometry>
+            <box size="0.01 0.05 0.03"/>
+          </geometry>
+        </visual>
+        <collision>
+          <origin xyz="0 0 0" rpy="0 0 0"/>
+          <geometry>
+            <box size="0.01 0.05 0.03"/>
+          </geometry>
+        </collision>
+        <inertial>
+          <mass value="0.300" />
+          <inertia
+            ixx="0.001" ixy="0" ixz="0"
+            iyy="0.001" iyz="0"
+            izz="0.01" />
+        </inertial>
+      </link>
+      <joint name="${prefix}_camera_joint" type="fixed">
+          <parent link="${origin_link}"/>
+          <child link="${prefix}_camera_link"/>
+          <origin rpy="${rpy}" xyz="${xyz}"/>
+      </joint>
+      <link name="${prefix}_lens_link"></link>
+      <joint name="${prefix}_lens_joint" type="fixed">
+          <parent link="${prefix}_camera_link"/>
+          <child link="${prefix}_lens_link"/>
+          <origin xyz="0 0 0" rpy="-1.57 0 -1.57"/>
+      </joint>
+          <!-- camera -->
+      <gazebo reference="${prefix}_camera_link">
+        <sensor type="depth" name="camera_link_sensor">
+          <!-- offset between camera_link and camera_depth_optical_link -->
+          <!-- additional mm offsets added through inspection -->
+          <pose>-0.001 -0.045 0.001 -0.000 0 1.57</pose>
+          <always_on>true</always_on>
+          <update_rate>15.0</update_rate>
+          <camera>
+            <horizontal_fov>${57.0*M_PI/180.0}</horizontal_fov>
+            <image>
+              <format>R8G8B8</format>
+              <width>640</width>
+              <height>480</height>
+            </image>
+            <clip>
+              <near>0.01</near>
+              <far>5</far>
+            </clip>
+          </camera>
+          <plugin name="kinect_camera" filename="libgazebo_ros_openni_kinect.so">
+            <alwaysOn>true</alwaysOn>
+            <updateRate>15.0</updateRate>
+            <cameraName>${prefix}_camera</cameraName>
+            <frameName>GT/${prefix}_lens_link</frameName>
+            <imageTopicName>${prefix}_camera/rgb/image_rect_color</imageTopicName>
+            <cameraInfoTopicName>${prefix}_camera/rgb/camera_info</cameraInfoTopicName>
+            <depthImageTopicName>${prefix}_camera/depth_registered/image_raw</depthImageTopicName>
+            <depthImageCameraInfoTopicName>${prefix}_camera/depth_registered/camera_info</depthImageCameraInfoTopicName>
+            <pointCloudTopicName>${prefix}_camera/depth/points</pointCloudTopicName>
+            <pointCloudCutoff>0.5</pointCloudCutoff>
+            <distortionK1>0.00000001</distortionK1>
+            <distortionK2>0.00000001</distortionK2>
+            <distortionK3>0.00000001</distortionK3>
+            <distortionT1>0.00000001</distortionT1>
+            <distortionT2>0.00000001</distortionT2>
+          </plugin>
+        </sensor>
+      </gazebo>
     </xacro:macro>
 </robot>

File: urdf/depth_camera_test.urdf.xacro (robot description, xacro)
@@ -2,5 +2,5 @@
 <robot name="roscontrol" xmlns:xacro="http://ros.org/wiki/xacro">
     <link name="base_link"></link>
-    <xacro:include filename="camera.urdf.xacro" ns="camera"/>
+    <xacro:include filename="depth_camera.urdf.xacro" ns="camera"/>
     <joint name="camera_joint" type="fixed">
         <parent link="base_link"/>

File: urdf/robot.urdf.xacro (robot description, xacro)
@@ -8,8 +8,8 @@
     </joint>
     <xacro:include filename="depth_camera.urdf.xacro"/>
-    <!--<xacro:kinect prefix="front" origin_link="base_link" xyz="0.15 0 0.25" rpy="0 0 0"/>
-    <xacro:kinect prefix="back" origin_link="base_link" xyz="-0.15 0 0.25" rpy="0 0 3.14"/>-->
+    <xacro:kinect prefix="front" origin_link="base_link" xyz="0.15 0 0.25" rpy="0 0 0"/>
+    <xacro:kinect prefix="back" origin_link="base_link" xyz="-0.15 0 0.25" rpy="0 0 3.14"/>
     <xacro:include filename="wide_camera.urdf.xacro"/>
-    <xacro:wide prefix="left" origin_link="base_link" xyz="0 -0.15 0.1" rpy="0 1.57 1.57"/>
-    <xacro:wide prefix="right" origin_link="base_link" xyz="0 0.15 0.1" rpy="1.57 1.57 0"/>
+    <xacro:wide prefix="left" origin_link="base_link" xyz="0 -0.15 0.1" rpy="0 0 -1.57"/>
+    <xacro:wide prefix="right" origin_link="base_link" xyz="0 0.15 0.1" rpy="0 0 1.57"/>
 </robot>

File: urdf/wide_camera.urdf.xacro (robot description, xacro)
@@ -1,6 +1,6 @@
 <?xml version="1.0"?>
 <robot name="chassis" xmlns:xacro="http://ros.org/wiki/xacro">
-    <xacro:property name="M_PI" value="3.1415926535897931" />
-    <xacro:macro name="wide" params="prefix origin_link xyz rpy">
+  <xacro:property name="M_PI" value="3.1415926535897931" />
+  <xacro:macro name="wide" params="prefix origin_link xyz rpy">
     <link name="${prefix}_camera_link">
       <visual>
@@ -35,5 +35,5 @@
         <origin xyz="0 0 0" rpy="-1.57 0 -1.57"/>
     </joint>
-<gazebo reference="${prefix}_camera_link">
+    <gazebo reference="${prefix}_camera_link">
         <sensor name="${prefix}_camera" type="wideanglecamera">
             <camera>
@@ -83,4 +83,4 @@
         </sensor>
     </gazebo>
-    </xacro:macro>
+  </xacro:macro>
 </robot>
