Commit message: tuned wheel a bit

File: urdf/chassis.urdf.xacro (robot description, xacro)
@@ -78,11 +78,11 @@
             <child link="${prefix}_${suffix}_roller"/>
             <origin xyz="${sin(theta)*roller_radius} ${roller_side_length*side} ${cos(theta)*roller_radius}" rpy="0 ${theta} 0"/>
-            <dynamics damping="0.00001" />
+            <dynamics damping="0.0001" />
         </joint>
         <!-- This block provides the simulator (Gazebo) with information on a few additional
         physical properties. See http://gazebosim.org/tutorials/?tut=ros_urdf for more-->
         <gazebo reference="${prefix}_${suffix}_roller">
-            <mu1 value="200.0"/>
-            <mu2 value="100.0"/>
+            <mu1 value="2000.0"/>
+            <mu2 value="1000.0"/>
             <kp value="10000000.0" />
             <kd value="1.0" />
@@ -122,5 +122,5 @@
             <kp value="10000000.0" />
             <kd value="1.0" />
-            <material>Gazebo/Grey</material>
+            <material>Gazebo/Green</material>
         </gazebo>
         <!-- This block connects the wheel joint to an actuator (motor), which informs both

Commit message: Make a loose facsimile of a V5 motor, spawn it on robot for testing
requires https://github.com/nilseuropa/gazebo_ros_motors in catkin workspace

File: urdf/chassis.urdf.xacro (robot description, xacro)
@@ -56,4 +56,28 @@
         <xacro:chassis_inertial mass="10"/>
     </link>
+    <link name="test_link">
+        <visual>
+            <origin xyz="0 0 0" rpy="0 0 0" />
+            <geometry>
+              <box size="0.05 0.05 0.03"/>
+            </geometry>
+            <material name="blue"/>
+        </visual>
+        <collision>
+            <origin xyz="0 0 0" rpy="0 0 0" />
+            <geometry>
+              <box size="0.05 0.05 0.03"/>
+            </geometry>
+        </collision>
+        <inertial>
+            <mass value="0.01" />
+            <inertia ixx="0.001" ixy="0.0" ixz="0.0" iyy="0.001" iyz="0.0" izz="0.001" />
+        </inertial>
+    </link>
+  <xacro:include filename="$(find gazebo_ros_motors)/xacro/dc_motor.xacro"/>
+  <xacro:dc_motor motor_name="top" parent_link="chassis_link" child_link="test_link">
+    <xacro:property name="params_yaml" value="$(find gazeboSimulation)/config/v5_motor.yaml"/>
+    <origin xyz="0 0 0.2" rpy="0 0 0"/>
+  </xacro:dc_motor>
     <xacro:macro name="roller" params="prefix suffix theta side">
         <link name="${prefix}_${suffix}_roller">

Commit message: got PID to work with v5 motors (just not well)

File: urdf/chassis.urdf.xacro (robot description, xacro)
@@ -75,9 +75,9 @@
         </inertial>
     </link>
-  <xacro:include filename="$(find gazebo_ros_motors)/xacro/dc_motor.xacro"/>
-  <xacro:dc_motor motor_name="top" parent_link="chassis_link" child_link="test_link">
-    <xacro:property name="params_yaml" value="$(find gazeboSimulation)/config/v5_motor.yaml"/>
-    <origin xyz="0 0 0.2" rpy="0 0 0"/>
-  </xacro:dc_motor>
+    <xacro:include filename="$(find gazebo_ros_motors)/xacro/dc_motor.xacro"/>
+    <xacro:dc_motor motor_name="top" parent_link="chassis_link" child_link="test_link">
+      <xacro:property name="params_yaml" value="$(find gazeboSimulation)/config/v5_motor.yaml"/>
+      <origin xyz="0 0 0.2" rpy="0 0 0"/>
+    </xacro:dc_motor>
     <xacro:macro name="roller" params="prefix suffix theta side">
         <link name="${prefix}_${suffix}_roller">

Commit message: robot is now fully pid

File: urdf/chassis.urdf.xacro (robot description, xacro)
@@ -1,4 +1,5 @@
 <?xml version="1.0"?>
 <robot name="chassis" xmlns:xacro="http://ros.org/wiki/xacro">
+    <xacro:include filename="$(find gazebo_ros_motors)/xacro/dc_motor.xacro"/>
     <xacro:property name="width" value="0.1" />
     <xacro:property name="leglen" value="0.05" />
@@ -56,28 +57,4 @@
         <xacro:chassis_inertial mass="10"/>
     </link>
-    <link name="test_link">
-        <visual>
-            <origin xyz="0 0 0" rpy="0 0 0" />
-            <geometry>
-              <box size="0.05 0.05 0.03"/>
-            </geometry>
-            <material name="blue"/>
-        </visual>
-        <collision>
-            <origin xyz="0 0 0" rpy="0 0 0" />
-            <geometry>
-              <box size="0.05 0.05 0.03"/>
-            </geometry>
-        </collision>
-        <inertial>
-            <mass value="0.01" />
-            <inertia ixx="0.001" ixy="0.0" ixz="0.0" iyy="0.001" iyz="0.0" izz="0.001" />
-        </inertial>
-    </link>
-    <xacro:include filename="$(find gazebo_ros_motors)/xacro/dc_motor.xacro"/>
-    <xacro:dc_motor motor_name="top" parent_link="chassis_link" child_link="test_link">
-      <xacro:property name="params_yaml" value="$(find gazeboSimulation)/config/v5_motor.yaml"/>
-      <origin xyz="0 0 0.2" rpy="0 0 0"/>
-    </xacro:dc_motor>
     <xacro:macro name="roller" params="prefix suffix theta side">
         <link name="${prefix}_${suffix}_roller">
@@ -131,4 +108,61 @@
                 </geometry>
             </collision>
+            <inertial>
+                <mass value="0.01" />
+                <inertia ixx="0.001" ixy="0.0" ixz="0.0" iyy="0.001" iyz="0.0" izz="0.001" />
+            </inertial>
+        </link>
+        <xacro:dc_motor motor_name="${prefix}_${suffix}_motor" parent_link="chassis_link" child_link="${prefix}_${suffix}_wheel">
+            <xacro:property name="params_yaml" value="$(find gazeboSimulation)/config/v5_motor.yaml"/>
+            <origin xyz="${baselen*reflect/3} ${.1*reflectX} -.05" rpy="0 0 0"/>
+        </xacro:dc_motor>
+        <gazebo reference="${prefix}_${suffix}_wheel">
+            <material>Gazebo/Green</material>
+        </gazebo>
+        <xacro:roller prefix="${prefix}_${suffix}" suffix="right_one" theta="${pi * ( 1/6)}" side="-1"/>
+        <xacro:roller prefix="${prefix}_${suffix}" suffix="right_two" theta="${pi * ( 2/6)}" side="-1"/>
+        <xacro:roller prefix="${prefix}_${suffix}" suffix="right_thr" theta="${pi * ( 3/6)}" side="-1"/>
+        <xacro:roller prefix="${prefix}_${suffix}" suffix="right_for" theta="${pi * ( 4/6)}" side="-1"/>
+        <xacro:roller prefix="${prefix}_${suffix}" suffix="right_fve" theta="${pi * ( 5/6)}" side="-1"/>
+        <xacro:roller prefix="${prefix}_${suffix}" suffix="right_six" theta="${pi * ( 6/6)}" side="-1"/>
+        <xacro:roller prefix="${prefix}_${suffix}" suffix="right_svn" theta="${pi * ( 7/6)}" side="-1"/>
+        <xacro:roller prefix="${prefix}_${suffix}" suffix="right_ate" theta="${pi * ( 8/6)}" side="-1"/>
+        <xacro:roller prefix="${prefix}_${suffix}" suffix="right_nne" theta="${pi * ( 9/6)}" side="-1"/>
+        <xacro:roller prefix="${prefix}_${suffix}" suffix="right_ten" theta="${pi * (10/6)}" side="-1"/>
+        <xacro:roller prefix="${prefix}_${suffix}" suffix="right_lvn" theta="${pi * (11/6)}" side="-1"/>
+        <xacro:roller prefix="${prefix}_${suffix}" suffix="right_wlv" theta="${pi * (12/6)}" side="-1"/>
+        <xacro:roller prefix="${prefix}_${suffix}" suffix="left_one" theta="${pi * ( 1/6) + ( pi / 12 )}" side="1"/>
+        <xacro:roller prefix="${prefix}_${suffix}" suffix="left_two" theta="${pi * ( 2/6) + ( pi / 12 )}" side="1"/>
+        <xacro:roller prefix="${prefix}_${suffix}" suffix="left_thr" theta="${pi * ( 3/6) + ( pi / 12 )}" side="1"/>
+        <xacro:roller prefix="${prefix}_${suffix}" suffix="left_for" theta="${pi * ( 4/6) + ( pi / 12 )}" side="1"/>
+        <xacro:roller prefix="${prefix}_${suffix}" suffix="left_fve" theta="${pi * ( 5/6) + ( pi / 12 )}" side="1"/>
+        <xacro:roller prefix="${prefix}_${suffix}" suffix="left_six" theta="${pi * ( 6/6) + ( pi / 12 )}" side="1"/>
+        <xacro:roller prefix="${prefix}_${suffix}" suffix="left_svn" theta="${pi * ( 7/6) + ( pi / 12 )}" side="1"/>
+        <xacro:roller prefix="${prefix}_${suffix}" suffix="left_ate" theta="${pi * ( 8/6) + ( pi / 12 )}" side="1"/>
+        <xacro:roller prefix="${prefix}_${suffix}" suffix="left_nne" theta="${pi * ( 9/6) + ( pi / 12 )}" side="1"/>
+        <xacro:roller prefix="${prefix}_${suffix}" suffix="left_ten" theta="${pi * (10/6) + ( pi / 12 )}" side="1"/>
+        <xacro:roller prefix="${prefix}_${suffix}" suffix="left_lvn" theta="${pi * (11/6) + ( pi / 12 )}" side="1"/>
+        <xacro:roller prefix="${prefix}_${suffix}" suffix="left_wlv" theta="${pi * (12/6) + ( pi / 12 )}" side="1"/>
+    </xacro:macro>
+    <xacro:wheel prefix="left" suffix="front"   reflect="1" reflectX="1"/>
+    <xacro:wheel prefix="left" suffix="back"   reflect="-1" reflectX="1"/>
+    <xacro:wheel prefix="right" suffix="front" reflect= "1" reflectX= "-1"/>
+    <xacro:wheel prefix="right" suffix="back" reflect= "-1" reflectX= "-1"/>
+<!--
+    <xacro:macro name="wheel" params="prefix suffix reflect reflectX">
+        <link name="${prefix}_${suffix}_wheel">
+            <visual>
+                <origin xyz="0 0 0" rpy="${pi/2} 0 0" />
+                <geometry>
+                    <cylinder radius="${wheeldiam/2}" length="${wheel_width}"/>
+                </geometry>
+                <material name="black"/>
+            </visual>
+            <collision>
+                <origin xyz="0 0 0" rpy="${pi/2} 0 0" />
+                <geometry>
+                    <cylinder radius="${wheeldiam/2}" length="${wheel_width}"/>
+                </geometry>
+            </collision>
             <xacro:roller_inertial mass="0.001"/>
         </link>
@@ -139,6 +173,4 @@
             <origin xyz="${baselen*reflect/3} ${.1*reflectX} -.05" rpy="0 0 0"/>
         </joint>
-        <!-- This block provides the simulator (Gazebo) with information on a few additional
-        physical properties. See http://gazebosim.org/tutorials/?tut=ros_urdf for more-->
         <gazebo reference="${prefix}_${suffix}_wheel">
             <mu1 value="200.0"/>
@@ -148,6 +180,4 @@
             <material>Gazebo/Green</material>
         </gazebo>
-        <!-- This block connects the wheel joint to an actuator (motor), which informs both
-        simulation and visualization of the robot -->
         <transmission name="${prefix}_${suffix}_wheel_trans">
             <type>transmission_interface/SimpleTransmission</type>
@@ -184,8 +214,5 @@
         <xacro:roller prefix="${prefix}_${suffix}" suffix="left_wlv" theta="${pi * (12/6) + ( pi / 12 )}" side="1"/>
     </xacro:macro>
-    <xacro:wheel prefix="left" suffix="front"  reflect= "1" reflectX="1"/>
-    <xacro:wheel prefix="left" suffix="back"   reflect="-1" reflectX="1"/>
-    <xacro:wheel prefix="right" suffix="front" reflect= "1" reflectX= "-1"/>
-    <xacro:wheel prefix="right" suffix="back"  reflect="-1" reflectX= "-1"/>
+    -->
     <!-- Gazebo plugin for ROS Control -->
     <gazebo>

Commit message: added real motors. tried figuring out a drive controller / odom but no
start from now and move to simulate motors

File: urdf/chassis.urdf.xacro (robot description, xacro)
@@ -1,4 +1,5 @@
 <?xml version="1.0"?>
 <robot name="chassis" xmlns:xacro="http://ros.org/wiki/xacro">
+    <xacro:include filename="$(find gazebo_ros_motors)/xacro/dc_motor.xacro"/>
     <xacro:property name="width" value="0.1" />
     <xacro:property name="leglen" value="0.05" />
@@ -107,32 +108,16 @@
                 </geometry>
             </collision>
-            <xacro:roller_inertial mass="0.001"/>
+            <inertial>
+                <mass value="0.01" />
+                <inertia ixx="0.001" ixy="0.0" ixz="0.0" iyy="0.001" iyz="0.0" izz="0.001" />
+            </inertial>
         </link>
-        <joint name="${prefix}_${suffix}_wheel_joint" type="continuous">
-            <axis xyz="0 1 0" />
-            <parent link="chassis_link"/>
-            <child link="${prefix}_${suffix}_wheel"/>
+        <xacro:dc_motor motor_name="${prefix}_${suffix}_motor" parent_link="chassis_link" child_link="${prefix}_${suffix}_wheel">
+            <xacro:property name="params_yaml" value="$(find simulation)/config/v5_motor.yaml"/>
             <origin xyz="${baselen*reflect/3} ${.1*reflectX} -.05" rpy="0 0 0"/>
-        </joint>
-        <!-- This block provides the simulator (Gazebo) with information on a few additional
-        physical properties. See http://gazebosim.org/tutorials/?tut=ros_urdf for more-->
+        </xacro:dc_motor>
         <gazebo reference="${prefix}_${suffix}_wheel">
-            <mu1 value="200.0"/>
-            <mu2 value="100.0"/>
-            <kp value="10000000.0" />
-            <kd value="1.0" />
             <material>Gazebo/Green</material>
         </gazebo>
-        <!-- This block connects the wheel joint to an actuator (motor), which informs both
-        simulation and visualization of the robot -->
-        <transmission name="${prefix}_${suffix}_wheel_trans">
-            <type>transmission_interface/SimpleTransmission</type>
-            <actuator name="${prefix}_${suffix}_wheel_motor">
-                <mechanicalReduction>1</mechanicalReduction>
-            </actuator>
-            <joint name="${prefix}_${suffix}_wheel_joint">
-                <hardwareInterface>VelocityJointInterface</hardwareInterface>
-            </joint>
-        </transmission>
         <xacro:roller prefix="${prefix}_${suffix}" suffix="right_one" theta="${pi * ( 1/6)}" side="-1"/>
         <xacro:roller prefix="${prefix}_${suffix}" suffix="right_two" theta="${pi * ( 2/6)}" side="-1"/>
@@ -160,9 +145,73 @@
         <xacro:roller prefix="${prefix}_${suffix}" suffix="left_wlv" theta="${pi * (12/6) + ( pi / 12 )}" side="1"/>
     </xacro:macro>
-    <xacro:wheel prefix="left" suffix="front"  reflect= "1" reflectX="1"/>
+    <xacro:wheel prefix="left" suffix="front"   reflect="1" reflectX="1"/>
     <xacro:wheel prefix="left" suffix="back"   reflect="-1" reflectX="1"/>
     <xacro:wheel prefix="right" suffix="front" reflect= "1" reflectX= "-1"/>
-    <xacro:wheel prefix="right" suffix="back"  reflect="-1" reflectX= "-1"/>
-    <!-- Gazebo plugin for ROS Control -->
+    <xacro:wheel prefix="right" suffix="back" reflect= "-1" reflectX= "-1"/>
+    <!--
+        <xacro:macro name="wheel" params="prefix suffix reflect reflectX">
+            <link name="${prefix}_${suffix}_wheel">
+                <visual>
+                    <origin xyz="0 0 0" rpy="${pi/2} 0 0" />
+                    <geometry>
+                        <cylinder radius="${wheeldiam/2}" length="${wheel_width}"/>
+                    </geometry>
+                    <material name="black"/>
+                </visual>
+                <collision>
+                    <origin xyz="0 0 0" rpy="${pi/2} 0 0" />
+                    <geometry>
+                        <cylinder radius="${wheeldiam/2}" length="${wheel_width}"/>
+                    </geometry>
+                </collision>
+                <xacro:roller_inertial mass="0.001"/>
+            </link>
+            <joint name="${prefix}_${suffix}_wheel_joint" type="continuous">
+                <axis xyz="0 1 0" />
+                <parent link="chassis_link"/>
+                <child link="${prefix}_${suffix}_wheel"/>
+                <origin xyz="${baselen*reflect/3} ${.1*reflectX} -.05" rpy="0 0 0"/>
+            </joint>
+            <gazebo reference="${prefix}_${suffix}_wheel">
+                <mu1 value="200.0"/>
+                <mu2 value="100.0"/>
+                <kp value="10000000.0" />
+                <kd value="1.0" />
+                <material>Gazebo/Green</material>
+            </gazebo>
+            <transmission name="${prefix}_${suffix}_wheel_trans">
+                <type>transmission_interface/SimpleTransmission</type>
+                <actuator name="${prefix}_${suffix}_wheel_motor">
+                    <mechanicalReduction>1</mechanicalReduction>
+                </actuator>
+                <joint name="${prefix}_${suffix}_wheel_joint">
+                    <hardwareInterface>VelocityJointInterface</hardwareInterface>
+                </joint>
+            </transmission>
+            <xacro:roller prefix="${prefix}_${suffix}" suffix="right_one" theta="${pi * ( 1/6)}" side="-1"/>
+            <xacro:roller prefix="${prefix}_${suffix}" suffix="right_two" theta="${pi * ( 2/6)}" side="-1"/>
+            <xacro:roller prefix="${prefix}_${suffix}" suffix="right_thr" theta="${pi * ( 3/6)}" side="-1"/>
+            <xacro:roller prefix="${prefix}_${suffix}" suffix="right_for" theta="${pi * ( 4/6)}" side="-1"/>
+            <xacro:roller prefix="${prefix}_${suffix}" suffix="right_fve" theta="${pi * ( 5/6)}" side="-1"/>
+            <xacro:roller prefix="${prefix}_${suffix}" suffix="right_six" theta="${pi * ( 6/6)}" side="-1"/>
+            <xacro:roller prefix="${prefix}_${suffix}" suffix="right_svn" theta="${pi * ( 7/6)}" side="-1"/>
+            <xacro:roller prefix="${prefix}_${suffix}" suffix="right_ate" theta="${pi * ( 8/6)}" side="-1"/>
+            <xacro:roller prefix="${prefix}_${suffix}" suffix="right_nne" theta="${pi * ( 9/6)}" side="-1"/>
+            <xacro:roller prefix="${prefix}_${suffix}" suffix="right_ten" theta="${pi * (10/6)}" side="-1"/>
+            <xacro:roller prefix="${prefix}_${suffix}" suffix="right_lvn" theta="${pi * (11/6)}" side="-1"/>
+            <xacro:roller prefix="${prefix}_${suffix}" suffix="right_wlv" theta="${pi * (12/6)}" side="-1"/>
+            <xacro:roller prefix="${prefix}_${suffix}" suffix="left_one" theta="${pi * ( 1/6) + ( pi / 12 )}" side="1"/>
+            <xacro:roller prefix="${prefix}_${suffix}" suffix="left_two" theta="${pi * ( 2/6) + ( pi / 12 )}" side="1"/>
+            <xacro:roller prefix="${prefix}_${suffix}" suffix="left_thr" theta="${pi * ( 3/6) + ( pi / 12 )}" side="1"/>
+            <xacro:roller prefix="${prefix}_${suffix}" suffix="left_for" theta="${pi * ( 4/6) + ( pi / 12 )}" side="1"/>
+            <xacro:roller prefix="${prefix}_${suffix}" suffix="left_fve" theta="${pi * ( 5/6) + ( pi / 12 )}" side="1"/>
+            <xacro:roller prefix="${prefix}_${suffix}" suffix="left_six" theta="${pi * ( 6/6) + ( pi / 12 )}" side="1"/>
+            <xacro:roller prefix="${prefix}_${suffix}" suffix="left_svn" theta="${pi * ( 7/6) + ( pi / 12 )}" side="1"/>
+            <xacro:roller prefix="${prefix}_${suffix}" suffix="left_ate" theta="${pi * ( 8/6) + ( pi / 12 )}" side="1"/>
+            <xacro:roller prefix="${prefix}_${suffix}" suffix="left_nne" theta="${pi * ( 9/6) + ( pi / 12 )}" side="1"/>
+            <xacro:roller prefix="${prefix}_${suffix}" suffix="left_ten" theta="${pi * (10/6) + ( pi / 12 )}" side="1"/>
+            <xacro:roller prefix="${prefix}_${suffix}" suffix="left_lvn" theta="${pi * (11/6) + ( pi / 12 )}" side="1"/>
+            <xacro:roller prefix="${prefix}_${suffix}" suffix="left_wlv" theta="${pi * (12/6) + ( pi / 12 )}" side="1"/>
+        </xacro:macro>
     <gazebo>
         <plugin name="gazebo_ros_control" filename="libgazebo_ros_control.so">
@@ -170,13 +219,14 @@
         </plugin>
         <plugin name="p3d_base_controller" filename="libgazebo_ros_p3d.so">
-          <alwaysOn>true</alwaysOn>
-          <updateRate>50.0</updateRate>
-          <bodyName>chassis_link</bodyName>
-          <topicName>ground_truth/state</topicName>
-          <gaussianNoise>0.01</gaussianNoise>
-          <frameName>world</frameName>
-          <xyzOffsets>0 0 0</xyzOffsets>
-          <rpyOffsets>0 0 0</rpyOffsets>
+            <alwaysOn>true</alwaysOn>
+            <updateRate>50.0</updateRate>
+            <bodyName>chassis_link</bodyName>
+            <topicName>ground_truth/state</topicName>
+            <gaussianNoise>0.01</gaussianNoise>
+            <frameName>world</frameName>
+            <xyzOffsets>0 0 0</xyzOffsets>
+            <rpyOffsets>0 0 0</rpyOffsets>
         </plugin>
     </gazebo>
+            -->
 </robot>

Commit message: wheels not spinning on correct axis

File: urdf/chassis.urdf.xacro (robot description, xacro)
@@ -115,5 +115,5 @@
         <xacro:dc_motor motor_name="${prefix}_${suffix}_motor" parent_link="chassis_link" child_link="${prefix}_${suffix}_wheel">
             <xacro:property name="params_yaml" value="$(find simulation)/config/v5_motor.yaml"/>
-            <origin xyz="${baselen*reflect/3} ${.1*reflectX} -.05" rpy="0 0 0"/>
+            <origin xyz="${baselen*reflect/3} ${.1*reflectX} -.05" rpy="0 1 0"/>
         </xacro:dc_motor>
         <gazebo reference="${prefix}_${suffix}_wheel">

Commit message: fixed the piece I couldnt figure out months ago

File: urdf/chassis.urdf.xacro (robot description, xacro)
@@ -113,7 +113,14 @@
             </inertial>
         </link>
-        <xacro:dc_motor motor_name="${prefix}_${suffix}_motor" parent_link="chassis_link" child_link="${prefix}_${suffix}_wheel">
+        <link name="${prefix}_${suffix}_shaft">
+        </link>
+        <joint name="${prefix}_${suffix}_shaft_joint" type="fixed">
+            <parent link="${prefix}_${suffix}_shaft"/>
+            <child link="${prefix}_${suffix}_wheel"/>
+            <origin xyz="0 0 0" rpy="${pi/2} 0 0"/>
+        </joint>
+        <xacro:dc_motor motor_name="${prefix}_${suffix}_motor" parent_link="chassis_link" child_link="${prefix}_${suffix}_shaft">
             <xacro:property name="params_yaml" value="$(find simulation)/config/v5_motor.yaml"/>
-            <origin xyz="${baselen*reflect/3} ${.1*reflectX} -.05" rpy="0 1 0"/>
+            <origin xyz="${baselen*reflect/3} ${.1*reflectX} -.05" rpy="${pi/2} 0 0"/>
         </xacro:dc_motor>
         <gazebo reference="${prefix}_${suffix}_wheel">
